File: Hardware/Make Files/Active/OBD2_SMS_GPRS.sch (KiCad schematic (older format))
At the start: 46 parts, among them P6 SMA, P7 SMA, P8 47553-1001, Q12 2N3904, Q13 2N3904, SW2 SW_PUSH_SMALL, SW3 SW_PUSH_SMALL, SW4 SW_PUSH_SMALL, SW5 SW_PUSH_SMALL, U15 SMF05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

Commit message: Some changes for V1.1
Making a backup point, I am planning to rename all the files to
V2X_xx.xx
Parts:
- removed C45, C46: dns, Capacitors_SMD:C_0603, symbol C
- removed C48, C50: 0, Capacitors_SMD:C_0603, symbol C
- removed L2, L4, L5, L6, L7, L8: dns, Capacitors_SMD:C_0805, symbol INDUCTOR_SMALL
- removed SW2, SW3, SW4, SW5: SW_PUSH_SMALL, Buttons_Switches_SMD:SW_SPST_FSMSM, symbol SW_PUSH_SMALL
- removed U15: SMF05, Housings_SOT-23_SOT-143_TSOT-6:SC-70-6_Handsoldering, symbol SMF05
- added A? (x2): ANTENNEA, symbol ANTENNEA
- added C? (x2): DNS, Capacitors_SMD:C_0603, symbol C
Connections:
- net labels added: GPS, GSM, GSM_DM, GSM_DP, GSM_VBUS
- wire segments 50 -> 49
- no-connect marks 10 -> 7
Other:
- note removed: "Button Input"
- moved on the sheet: C43, C44, C49, L1, L3, R63, R64, W1, W2
