File: Hardware/Make Files/Active/_autosave-V2X_SEQ.kicad_pcb (KiCad board)
At the start: 2 copper layers, 263 parts, among them CON1 AVR-PDI-6, IC1 ATXMEGA16A4U-A, J1 DB9, P1 47553-1001, P10 Board Mount 2, P11 Ficudial2, P12 Board Mount 3, P13 Ficudial3, P14 5V0_OUT, P15 Board Mount 4, P16 Ficudial4, P17 CUR_SEN, P18 CUR_SEN, P19 CUR_SEN, P2 SMA, P20 Jumper 1, P21 Jumper 2, P22 CONN_02X04, P23 Jumper 3, P24 Jumper 4, P25 CONN_02X08, P26 CONN_02X08, P3 SMA, P5 NVM_RST, P6 Board Mount 1, P7 Ficudial1, P8 Open Source, P9 USB_u, Q1 2N7000, Q10 2N3904, Q11 IRF9335, Q12 IRF9335, Q13 BSS84, Q14 IRF9335, Q15 2N7000, Q16 2N7000, Q17 2N7000, Q18 2N7000, Q19 2N7000, Q2 BSS84, Q3 BSS84, Q4 BSS84, Q5 3906, Q6 2N3904, Q7 2N7000, Q8 2N3904, Q9 2N3904, SW1 SPST, SW2 SW_PUSH, U1 FT4232H, U10 MCP2551, U11 XRP6124, U12 SLG59M, U14 XRP6124, U15 SLG59M, U16 SLG59M, U17 XRP6124, U18 SLG59M, U19 ADXL345, U2 93C46, U20 USB2242, U21 74LS126, U22 74HC595, U23 74HC595, U3 MMQA5V6T3G, U4 SIM5320, U5 ESDAxxSC6, U6 ESDAxxSC6, U7 STN1110, U8 LM339, U9 LM317, X1 12MHz, X2 16MHz, X3 24MHz

Commit message: Build pass of main V2X board
ready to verify
Parts:
- moved R34 151.3 mm to (170.0, 101.5), turned to 270 degrees
- moved R44 145.5 mm to (165.0, 101.5), turned to 90 degrees
- moved R57 143.8 mm to (152.5, 104.5)
- moved D9 141.8 mm to (162.5, 101.5), turned to 90 degrees
- moved R24 127.5 mm to (165.0, 97.0), turned to 90 degrees
- moved R32 127.0 mm to (170.0, 97.0), turned to 270 degrees
- moved R25 126.8 mm to (167.5, 97.0), turned to 270 degrees
- moved U9 119.4 mm to (157.0, 101.0)
- moved U7 111.6 mm to (213.5, 131.5)
- moved R42 65.2 mm to (163.5, 115.0), turned to 270 degrees
- moved C29 46.2 mm to (152.2, 142.2)
- moved C32 46.2 mm to (99.5, 137.5)
- moved C33 46.2 mm to (99.5, 135.0)
- moved C37 46.2 mm to (111.0, 137.0)
- moved C38 46.2 mm to (119.0, 138.8)
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Routing:
- net 5V0_B: track 56.9 -> 71.5 mm, vias 0 -> 1
- net GND: track 8.43 -> 18.5 mm, vias 5 -> 11
- net 5V0_EN: track 0.00 -> 9.33 mm
- net Net-(C44-Pad1): track 0.00 -> 8.89 mm, vias 0 -> 1
- net 12V0_B: track 23.5 -> 32.3 mm, vias 1 -> 3
- net Net-(C44-Pad2): track 0.00 -> 8.17 mm
- net Net-(Q11-Pad1): track 0.00 -> 4.88 mm, vias 0 -> 1
- net 5V0_A: track 0.00 -> 3.38 mm
- added copper zone on F.Cu, net 12V0_B
- added copper zone on F.Cu, net Net-(C44-Pad1)
- added copper zone on F.Cu, net Net-(D12-Pad1)
