File: Hardware/Make Files/Active/V2X_CTRL.sch (KiCad schematic (older format))
At the start: 8 parts

Commit message: Saving V1.1 as archive.
We are trying a new architecture where the FTDI can be removed. making a
backup spot
Parts:
- removed C?: 1U, symbol C
- removed FB?: FILTER, symbol FILTER
- removed R? (x2): 4K7, symbol R
- added C64, C65, C66, C67, C68: 100N, symbol C
- added C69: 1U, symbol C
- added D16: RED, LEDs:LED-0805, symbol LED
- added D17: BLUE, LEDs:LED-0805, symbol LED
- added FB6: FILTER, symbol FILTER
- added Q16, Q17, Q18: 2N7000, symbol Q_NMOS_SGD
- added R80: 0, Resistors_SMD:R_0603, symbol R
- added R81, R82: DNS, Resistors_SMD:R_0603, symbol R
- added R83: 330, Resistors_SMD:R_0603, symbol R
- added R84: 100, Resistors_SMD:R_0603, symbol R
- added R86, R87, R89: 10K, Resistors_SMD:R_0603, symbol R
- added U19: 74LS126, symbol 74LS126
- added U20, U21: 74HC595, symbol 74HC595
- gave numbers to parts that had none: 4
Connections:
- net labels added: 3V3_A, 3V3_B_EN, 3V3_C_EN, 3V3_D, 3V3_D_EN, 5V0_B_EN, 5V0_B_OUT, ACCEL_RXD, ACCEL_TXD, ACL_INT1, ACL_INT2, BUTTON, CAN_RXD, CAN_RXD_BUF, CAN_RXD_FTDI, CAN_RXD_PS, CAN_RXD_PS_BUF, CAN_TXD, FTDI_RESET, HUB_SCL, HUB_SDA, HUB_STATUS, HUB_SUSP, PC_LED1, PC_LED2, PC_WAKE, SIM_DTR, SIM_NET, SIM_PWR, SIM_PWR_ON, SIM_RF_OFF, SIM_RI, SIM_RXD, SIM_TXD, SIM_VBUS, SR_CLEAR, SR_LATCH, VCC, ~HUB_RESET, ~SIM_PWR_ON, ~SIM_RESET
- net labels removed: 3V3_ADC, 3V3_CONST, 5V0, 5V0_OUT, CAN_POWERDOWN, GPIO_1, GPIO_40, GPRS_EN, GPRS_RESET, HOST_5V0, MC_BUTTON, MD_LED1, MD_LED2, MD_LED3, STN_RXD_BUF, STN_TXD, UART_RI, UART_RXD_BUF, UART_TXD
- wire segments 19 -> 42
- no-connect marks 0 -> 1
Other:
- note added: "HUB /RESET\nELM/STN /Reset\nELM/STN /Sleep\nSIM Module "Power On"\nSIM Module /Reset\nSIM "Airplane Mode"\nSIM USB detect\nFTDI USB detect /RESET"
- note added: "HUB Serial Data I2C/SMB\nHUB Serial Clock I2C/SMB\nAccel Stream RXD to FTDI\nAccel Stream TXD to FTDI"
- note added: "Host Power Short Circuit detect\n\nCAN Ctrl RXD from PWRSEQ\nCAN Ctrl RXD from FTDI"
- note added: "PWRSEQ 3V3 Enable\nHUB/FTDI 3V3 Enable\nCAN 3V3 Enable\nAccel 3V3 Enable\n4V1 Power Supply Enable\n5V0 Power Supply Enable (CAN)\n5V0 Host Enable \n"
- note added: "PWRSEQ LED1 PWM Output\nPWRSEQ LED2 PWM Output\nSIM TXD to PWRSEQ and FTDI\nSIM RXD to PWRSEQ Buffer\n\nButton (pwr/soft) input\nCAN TXD to PWRSEQ and FTDI\nCAN RXD to PWRSEQ Buffer"
- note added: "PWRSEQ Reset/PDI_CLK\nPWRSEQ PDI Data"
- note added: "Power Ctrl Programing port"
- note added: "SIM Network Status Input\nSIM Power status Input\nSIMCARD (insterted) detect input\nSIM Host Wake-up input\nAccelerometer Interupt 1 input\nAccelerometer Interupt 2 input\nHUB Power State Status input\nHUB Suspend state input"
- note added: "Serial shift registers Outputs:\nAccelerometer data on SPI just passes \nthrough into the bit bucket until \nSR_LATCH is clocked high\nThe Accelerometer ignores the \nshift data while PC_SS is high\nSR_CLEAR + SR_LATCH sets all \noutputs to 0, default safe boot state."
- note added: "Shift Register clear outputs\nShift Register latch serial data \nPWRSEQ RXD to FTDI\nPWRSEQ TXD to FTDI\nAccelerometer SPI Chip Select\nShift Register Data and SPI Data OUT\nAccelerometer SPI Data IN\nShift Register and Acceleromter Clock"
- note added: "Short Circuit Detection\n5V0_USB is post poly fuse\nSample using A2D \n(maybe logic level for simplier detection)\nLow voltage (<2.4V) indicates\nfuse is set, host is short circuit.\nA value that is too high might \nindicate the Host is not attached."
- note added: "Turns the Negative\nPower-On" pulse\nto a positive pulse"
- note removed: "GSM ENABLE\nGSM RESET\nGSM_POWER_STAT\nGSM_NETWORK_STAT\nSIM CARD DETECT\nRING INDICATOR FROM GSM"
- note removed: "HOST->FTDI Serial Tx\nHOST->FTDI Serial Rx\nGSM->FTDI Snoop\n\nGSM Ring In indicator\nStatus LED 1\nStatus LED 2\nStatus LED 3\n"
- note removed: "MC_PROG\nMC_PROG\nMC_PROG"
- note removed: "OBD RESET\nOBD SLEEP\nOBD POWERDOWN STATUS"
- note removed: "Power and Control Sequencer"
- note removed: "Short Circuit Detection\n5V0_USB is post poly fuse\nLow voltage (<2.4V) indicates\nfuse is set, host is short circuit\nor off."
- note removed: "System Power button\n3V3_EN\n4V1_EN\n5V0_EN\n\n\n\nHost Short Circuit Detectioin"
- moved on the sheet: IC1, R85, R88

Commit message: V1.2 mostly done
BOM is integrated and creates mouser orders
Parts:
- removed C64: 100N, symbol C
- removed Q16: 2N7000, symbol Q_NMOS_SGD
- removed R83: 330, Resistors_SMD:R_0603, symbol R
- removed R85: 4K7, symbol R
- removed unit 2 of U19
- removed U21: 74HC595, symbol 74HC595
- added C70: 1U, symbol C
- added P20: CONN_02X04, symbol CONN_02X04
- added P?: Jumper 1, Mounting_Holes:MountingHole_3mm, symbol CONN_01X01
- added P?: Jumper 2, Mounting_Holes:MountingHole_3mm, symbol CONN_01X01
- added P?: Jumper 3, Mounting_Holes:MountingHole_3mm, symbol CONN_01X01
- added P?: Jumper 4, Mounting_Holes:MountingHole_3mm, symbol CONN_01X01
- added Q18: 2N7000, symbol Q_NMOS_SGD
- added R90: 330, Resistors_SMD:R_0603, symbol R
- added R93: 47K, Resistors_SMD:R_0603, symbol R
- added unit 2 of U21
- added U23: 74HC595, symbol 74HC595
- C65, C66, C67, C68: footprint (none) -> Capacitors_SMD:C_0603; Mouse PN (none) -> 810-C1608X7R1E104K
- C69: value 1U -> 100N; footprint (none) -> Capacitors_SMD:C_0603; Mouse PN (none) -> 810-C1608X7R1E104K
- CON1: Mouse PN (none) -> 571-5-146130-2
- D16: Mouse PN (none) -> 720-LSR976-NR-1
- D17: Mouse PN (none) -> 710-150080BS75000
- FB6: value FILTER -> 220; footprint (none) -> Capacitors_SMD:C_0805; Mouse PN (none) -> 810-MPZ1608S221ATA00
- IC1: Mouse PN (none) -> 556-ATXMEGA16A4U-AU
- Q16: renamed from Q18; Mouse PN (none) -> 512-2N7002K
- Q17: Mouse PN (none) -> 512-2N7002K
- R84: renamed from R80; value 0 -> DNS
- R85: renamed from R81; value DNS -> 0; Mouse PN (none) -> 71-CRCW0603-0-E3
- R87: Mouse PN (none) -> 71-CRCW0603-10K-E3
- R88: value 4K7 -> 47K; footprint (none) -> Resistors_SMD:R_0603; Mouse PN (none) -> 71-CRCW0603-47K-E3
- R89: value 10K -> 47K; Mouse PN (none) -> 71-CRCW0603-47K-E3
- R91: renamed from R84; value 100 -> 220; Mouse PN (none) -> 71-CRCW0603-220-E3
- R92: renamed from R86; value 10K -> 47K; Mouse PN (none) -> 71-CRCW0603-47K-E3
- U21: renamed from U19; Mouse PN (none) -> 863-MC74HC126ADR2G
- U22: renamed from U20; Mouse PN (none) -> 771-74HC595D-Q100
- renumbered R82 to R86
Connections:
- net labels added: 5V0_A, 5V0_C_EN, FTDI_DM, FTDI_DP, SEQ_BUTTON, SEQ_LED1, SEQ_LED2, SEQ_MISO, SEQ_MOSI, SEQ_RESET, SEQ_RXD, SEQ_RXD_DM, SEQ_SCK, SEQ_SS, SEQ_TXD, SEQ_TXD_DP, SEQ_WAKE, USB_INT_DM, USB_INT_DP, ~FTDI_RESET
- net labels removed: BUTTON, FTDI_RESET, PC_MISO, PC_MOSI, PC_RXD, PC_SCK, PC_SS, PC_TXD, PC_WAKE
- no-connect marks 1 -> 6
Other:
- note added: "3V3 Power Supply Enable (SEQ)\nHUB/FTDI 3V3 Enable\nCAN 3V3 Enable\nAccel 3V3 Enable\n4V1 Power Supply Enable (SIM)\n5V0 Power Supply Enable (LEDs)\n5V0 HOST Enable \n5V0 CAN Enable"
- note added: "JUMPERS = 1-3, 2-4, 5-7, 6-8\nFTDI is USB with FTDI to SEQ control channel open\n\nJUMPERS = 3-5, 4-6\nAtmel is USB and FTDI disabled"
- note added: "PDI Programing port"
- note added: "Power-On" negative pulse -> a SR positive pulse\nSo default SR state doesn't false start SIM module"
- note added: "SEQ LED1 PWM Output\nSEQ LED2 PWM Output\nSIM TXD to PWRSEQ and FTDI\nSIM RXD to PWRSEQ Buffer\n\nButton (pwr/soft) input\nSEQ RXD to FTDI\nSEQ TXD to FTDI"
- note added: "SEQ Reset/PDI_CLK\nSEQ PDI Data"
- note added: "Serial shift registers Outputs:\nSR_CLEAR + SR_LATCH sets all outputs to 0, default\nsafe boot state. Accelerometer data on SPI just passes\nthrough into the bit bucket until R_LATCH is clocked.\nThe Accelerometer ignores the shift data while SEQ_SS is high.\n"
- note added: "Shift Register clear outputs\nShift Register latch serial data \nCAN TXD to PWRSEQ and FTDI\nCAN RXD to PWRSEQ Buffer\nAccelerometer SPI Chip Select\nShift Register Data and SPI Data OUT\nAccelerometer SPI Data IN\nShift Register and Acceleromter Clock"
- note removed: "MC_PROG"
- note removed: "PWRSEQ 3V3 Enable\nHUB/FTDI 3V3 Enable\nCAN 3V3 Enable\nAccel 3V3 Enable\n4V1 Power Supply Enable\n5V0 Power Supply Enable (CAN)\n5V0 Host Enable \n"
- note removed: "PWRSEQ LED1 PWM Output\nPWRSEQ LED2 PWM Output\nSIM TXD to PWRSEQ and FTDI\nSIM RXD to PWRSEQ Buffer\n\nButton (pwr/soft) input\nCAN TXD to PWRSEQ and FTDI\nCAN RXD to PWRSEQ Buffer"
- note removed: "PWRSEQ Reset/PDI_CLK\nPWRSEQ PDI Data"
- note removed: "Power Ctrl Programing port"
- note removed: "Serial shift registers Outputs:\nAccelerometer data on SPI just passes \nthrough into the bit bucket until \nSR_LATCH is clocked high\nThe Accelerometer ignores the \nshift data while PC_SS is high\nSR_CLEAR + SR_LATCH sets all \noutputs to 0, default safe boot state."
- note removed: "Shift Register clear outputs\nShift Register latch serial data \nPWRSEQ RXD to FTDI\nPWRSEQ TXD to FTDI\nAccelerometer SPI Chip Select\nShift Register Data and SPI Data OUT\nAccelerometer SPI Data IN\nShift Register and Acceleromter Clock"
- note removed: "Turns the Negative\nPower-On" pulse\nto a positive pulse"
- moved on the sheet: D16, D17, Q16, R91, R92, U21A, U22

Commit message: V2X v1.2 sch and bom
Made changes to the schematic to V1.2 (remove FTDI possibly) and
integrade the BOM information into the sch
Parts:
- gave numbers to parts that had none: 4
- renumbered C65 to C59, C66 to C60, C67 to C61, C68 to C62, C69 to C63, C70 to C64, P20 to P22
Other:
- moved on the sheet: Q16, R87
Changed lines of the file:
@@
 Text GLabel 5150 1700 2    60   Input ~ 0
 SIMCARD
-Text GLabel 6650 3950 2    60   Input ~ 0
+Text GLabel 6650 4000 2    60   Input ~ 0
 ~SIM_PWR_ON
 Text GLabel 2500 6950 2    60   Input ~ 0
@@
 SEQ_LED2
 $Comp
-L GND #PWR0133
+L GND #PWR138
 U 1 1 55F86E9C
 P 4100 3900
-F 0 "#PWR0133" H 4100 3650 50  0001 C CNN
+F 0 "#PWR138" H 4100 3650 50  0001 C CNN
 F 1 "GND" H 4100 3750 50  0000 C CNN
 F 2 "" H 4100 3900 60  0000 C CNN
@@
 	8900 5850 8900 5950
 $Comp
-L GND #PWR0134
+L GND #PWR142
 U 1 1 55F86EC1
 P 8900 6250
-F 0 "#PWR0134" H 8900 6000 50  0001 C CNN
+F 0 "#PWR142" H 8900 6000 50  0001 C CNN
 F 1 "GND" H 8900 6100 50  0000 C CNN
 F 2 "" H 8900 6250 60  0000 C CNN
@@
 PDI
 $Comp
-L GND #PWR0135
+L GND #PWR140
 U 1 1 55F86EF0
 P 10050 4850
-F 0 "#PWR0135" H 10050 4600 50  0001 C CNN
+F 0 "#PWR140" H 10050 4600 50  0001 C CNN
 F 1 "GND" H 10050 4700 50  0000 C CNN
 F 2 "" H 10050 4850 60  0000 C CNN
@@
 5V0_B_EN
 $Comp
-L GND #PWR0136
+L GND #PWR141
 U 1 1 55FA434A
 P 1100 5750
-F 0 "#PWR0136" H 1100 5500 50  0001 C CNN
+F 0 "#PWR141" H 1100 5500 50  0001 C CNN
 F 1 "GND" H 1100 5600 50  0000 C CNN
 F 2 "" H 1100 5750 60  0000 C CNN
@@
 $EndComp
 $Comp
-L GND #PWR0137
+L GND #PWR145
 U 1 1 55FA46C8
 P 1100 7150
-F 0 "#PWR0137" H 1100 6900 50  0001 C CNN
+F 0 "#PWR145" H 1100 6900 50  0001 C CNN
 F 1 "GND" H 1100 7000 50  0000 C CNN
 F 2 "" H 1100 7150 60  0000 C CNN
@@
 Text Notes 5900 2700 0    69   ~ 0
 Host Power Short Circuit detect\n\nCAN Ctrl RXD from PWRSEQ\nCAN Ctrl RXD from FTDI
-Text Notes 650  4950 0    69   ~ 0
+Text Notes 700  4800 0    69   ~ 0
 Serial shift registers Outputs:\nSR_CLEAR + SR_LATCH sets all outputs to 0, default\nsafe boot state. Accelerometer data on SPI just passes\nthrough into the bit bucket until R_LATCH is clocked.\nThe Accelerometer ignores the shift data while SEQ_SS is high.\n
 Text GLabel 2500 7250 2    60   Input ~ 0
@@
 $EndComp
 $Comp
-L GND #PWR0138
+L GND #PWR143
 U 1 1 55FD726F
 P 5600 7100
-F 0 "#PWR0138" H 5600 6850 50  0001 C CNN
+F 0 "#PWR143" H 5600 6850 50  0001 C CNN
 F 1 "GND" H 5600 6950 50  0000 C CNN
 F 2 "" H 5600 7100 60  0000 C CNN
@@
 $EndComp
 $Comp
-L GND #PWR0139
+L GND #PWR146
 U 1 1 55FD7284
 P 5250 7250
-F 0 "#PWR0139" H 5250 7000 50  0001 C CNN
+F 0 "#PWR146" H 5250 7000 50  0001 C CNN
 F 1 "GND" H 5250 7100 50  0000 C CNN
 F 2 "" H 5250 7250 60  0000 C CNN
@@
 $EndComp
 $Comp
-L GND #PWR0140
+L GND #PWR147
 U 1 1 55FD7672
 P 6150 7250
-F 0 "#PWR0140" H 6150 7000 50  0001 C CNN
+F 0 "#PWR147" H 6150 7000 50  0001 C CNN
 F 1 "GND" H 6150 7100 50  0000 C CNN
 F 2 "" H 6150 7250 60  0000 C CNN
@@
 PC_LED2
 $Comp
-L GND #PWR0141
+L GND #PWR144
 U 1 1 55FD7660
 P 6500 7100
-F 0 "#PWR0141" H 6500 6850 50  0001 C CNN
+F 0 "#PWR144" H 6500 6850 50  0001 C CNN
 F 1 "GND" H 6500 6950 50  0000 C CNN
 F 2 "" H 6500 7100 60  0000 C CNN
@@
 L Q_NMOS_SGD Q16
 U 1 1 55FE0BA7
-P 6300 4350
-F 0 "Q16" H 6200 4450 50  0000 R CNN
-F 1 "2N7000" H 6300 4200 50  0000 R CNN
-F 2 "" H 6500 4450 29  0000 C CNN
-F 3 "http://www.mouser.com/ds/2/149/2N7002K-102052.pdf" H 6300 4350 60  0001 C CNN
-F 4 "512-2N7002K" H 6300 4350 60  0001 C CNN "Mouse PN"
-	1    6300 4350
-	1    0    0    -1
-$EndComp
-$Comp
-L GND #PWR0142
+P 6300 4400
+F 0 "Q16" H 6200 4500 50  0000 R CNN
+F 1 "2N7000" H 6300 4250 50  0000 R CNN
+F 2 "" H 6500 4500 29  0000 C CNN
+F 3 "http://www.mouser.com/ds/2/149/2N7002K-102052.pdf" H 6300 4400 60  0001 C CNN
+F 4 "512-2N7002K" H 6300 4400 60  0001 C CNN "Mouse PN"
+	1    6300 4400
+	1    0    0    -1
+$EndComp
+$Comp
+L GND #PWR139
 U 1 1 55FE1020
-P 6400 4550
-F 0 "#PWR0142" H 6400 4300 50  0001 C CNN
-F 1 "GND" H 6400 4400 50  0000 C CNN
-F 2 "" H 6400 4550 60  0000 C CNN
-F 3 "" H 6400 4550 60  0000 C CNN
-	1    6400 4550
+P 6400 4600
+F 0 "#PWR139" H 6400 4350 50  0001 C CNN
+F 1 "GND" H 6400 4450 50  0000 C CNN
+F 2 "" H 6400 4600 60  0000 C CNN
+F 3 "" H 6400 4600 60  0000 C CNN
+	1    6400 4600
 	1    0    0    -1
 $EndComp
@@
 HUB_STATUS
 Wire Wire Line
-	6650 4150 6650 3950
+	6650 4200 6650 4000
 Text GLabel 5150 2200 2    69   Input ~ 0
 HUB_SUSP
@@
 Connection ~ 10550 750
 $Comp
-L GND #PWR0143
+L GND #PWR137
 U 1 1 56006FBB
 P 10550 1100
-F 0 "#PWR0143" H 10550 850 50  0001 C CNN
+F 0 "#PWR137" H 10550 850 50  0001 C CNN
 F 1 "GND" H 10550 950 50  0000 C CNN
 F 2 "" H 10550 1100 60  0000 C CNN
@@
 NoConn ~ 2500 7450
 Wire Wire Line
-	6400 4150 6750 4150
-Text GLabel 6100 4350 0    60   Input ~ 0
+	6400 4200 6750 4200
+Text GLabel 6100 4400 0    60   Input ~ 0
 SIM_PWR_ON
 Text GLabel 2500 6850 2    60   Input ~ 0
@@
 Text GLabel 2500 5150 2    69   Input ~ 0
 3V3_EN
-Connection ~ 6650 4150
+Connection ~ 6650 4200
 Wire Wire Line
 	8400 750  9750 750
@@
 Connection ~ 9000 750
 $Comp
-L GND #PWR0144
+L GND #PWR134
 U 1 1 560285A0
 P 9000 1100
-F 0 "#PWR0144" H 9000 850 50  0001 C CNN
+F 0 "#PWR134" H 9000 850 50  0001 C CNN
 F 1 "GND" H 9000 950 50  0000 C CNN
 F 2 "" H 9000 1100 60  0000 C CNN
@@
 $EndComp
 $Comp
-L GND #PWR0145
+L GND #PWR135
 U 1 1 560285F6
 P 9300 1100
-F 0 "#PWR0145" H 9300 850 50  0001 C CNN
+F 0 "#PWR135" H 9300 850 50  0001 C CNN
 F 1 "GND" H 9300 950 50  0000 C CNN
 F 2 "" H 9300 1100 60  0000 C CNN
@@
 $EndComp
 $Comp
-L GND #PWR0146
+L GND #PWR136
 U 1 1 5602864C
 P 9600 1100
-F 0 "#PWR0146" H 9600 850 50  0001 C CNN
+F 0 "#PWR136" H 9600 850 50  0001 C CNN
 F 1 "GND" H 9600 950 50  0000 C CNN
 F 2 "" H 9600 1100 60  0000 C CNN
@@
 Connection ~ 9150 750
 $Comp
-L VCC #PWR0147
+L VCC #PWR131
 U 1 1 56029609
 P 9150 700
-F 0 "#PWR0147" H 9150 550 50  0001 C CNN
+F 0 "#PWR131" H 9150 550 50  0001 C CNN
 F 1 "VCC" H 9150 850 50  0000 C CNN
 F 2 "" H 9150 700 60  0000 C CNN
@@
 Connection ~ 8750 750
 $Comp
-L GND #PWR0148
+L GND #PWR133
 U 1 1 5602C4DB
 P 8750 1100
-F 0 "#PWR0148" H 8750 850 50  0001 C CNN
+F 0 "#PWR133" H 8750 850 50  0001 C CNN
 F 1 "GND" H 8750 950 50  0000 C CNN
 F 2 "" H 8750 1100 60  0000 C CNN
@@
 $EndComp
 $Comp
-L GND #PWR0149
+L GND #PWR132
 U 1 1 5602C537
 P 8450 1100
-F 0 "#PWR0149" H 8450 850 50  0001 C CNN
+F 0 "#PWR132" H 8450 850 50  0001 C CNN
 F 1 "GND" H 8450 950 50  0000 C CNN
 F 2 "" H 8450 1100 60  0000 C CNN
@@
 Text GLabel 10050 4650 2    60   Input ~ 0
 3V3_A
-Text GLabel 7050 4150 2    60   Input ~ 0
+Text GLabel 7050 4200 2    60   Input ~ 0
 3V3_A
 Text GLabel 9550 2600 0    60   Input ~ 0
@@
 USB_INT_DP
 $Comp
-L CONN_02X04 P20
+L CONN_02X04 P22
 U 1 1 56037434
 P 9100 3050
-F 0 "P20" H 9100 3300 50  0000 C CNN
+F 0 "P22" H 9100 3300 50  0000 C CNN
 F 1 "CONN_02X04" H 9100 2800 50  0000 C CNN
 F 2 "" H 9100 1850 60  0000 C CNN
@@
 	7950 1400 11200 1400
 $Comp
-L C C65
+L C C59
 U 1 1 56052557
 P 8450 950
-F 0 "C65" H 8475 1050 50  0000 L CNN
+F 0 "C59" H 8475 1050 50  0000 L CNN
 F 1 "100N" H 8475 850 50  0000 L CNN
 F 2 "Capacitors_SMD:C_0603" H 8488 800 30  0001 C CNN
@@
 $EndComp
 $Comp
-L C C66
+L C C60
 U 1 1 56052E12
 P 8750 950
-F 0 "C66" H 8775 1050 50  0000 L CNN
+F 0 "C60" H 8775 1050 50  0000 L CNN
 F 1 "100N" H 8775 850 50  0000 L CNN
 F 2 "Capacitors_SMD:C_0603" H 8788 800 30  0001 C CNN
@@
 $EndComp
 $Comp
-L C C67
+L C C61
 U 1 1 56052E7D
 P 9000 950
-F 0 "C67" H 9025 1050 50  0000 L CNN
+F 0 "C61" H 9025 1050 50  0000 L CNN
 F 1 "100N" H 9025 850 50  0000 L CNN
 F 2 "Capacitors_SMD:C_0603" H 9038 800 30  0001 C CNN
@@
 $EndComp
 $Comp
-L C C68
+L C C62
 U 1 1 56052EE9
 P 9300 950
-F 0 "C68" H 9325 1050 50  0000 L CNN
+F 0 "C62" H 9325 1050 50  0000 L CNN
 F 1 "100N" H 9325 850 50  0000 L CNN
 F 2 "Capacitors_SMD:C_0603" H 9338 800 30  0001 C CNN
@@
 $EndComp
 $Comp
-L C C69
+L C C63
 U 1 1 56052F58
 P 9600 950
-F 0 "C69" H 9625 1050 50  0000 L CNN
+F 0 "C63" H 9625 1050 50  0000 L CNN
 F 1 "100N" H 9625 850 50  0000 L CNN
 F 2 "Capacitors_SMD:C_0603" H 9638 800 30  0001 C CNN
@@
 $EndComp
 $Comp
-L C C70
+L C C64
 U 1 1 56059C07
 P 10550 950
-F 0 "C70" H 10575 1050 50  0000 L CNN
+F 0 "C64" H 10575 1050 50  0000 L CNN
 F 1 "1U" H 10575 850 50  0000 L CNN
 F 2 "" H 10588 800 30  0000 C CNN
@@
 L R R87
 U 1 1 5605AFDD
-P 6900 4150
-F 0 "R87" V 6980 4150 50  0000 C CNN
-F 1 "10K" V 6900 4150 50  0000 C CNN
-F 2 "Resistors_SMD:R_0603" V 6830 4150 30  0001 C CNN
-F 3 "http://www.mouser.com/ds/2/427/dcrcwe3-109170.pdf" H 6900 4150 30  0001 C CNN
-F 4 "71-CRCW0603-10K-E3" H 6900 4150 60  0001 C CNN "Mouse PN"
-	1    6900 4150
+P 6900 4200
+F 0 "R87" V 6980 4200 50  0000 C CNN
+F 1 "10K" V 6900 4200 50  0000 C CNN
+F 2 "Resistors_SMD:R_0603" V 6830 4200 30  0001 C CNN
+F 3 "http://www.mouser.com/ds/2/427/dcrcwe3-109170.pdf" H 6900 4200 30  0001 C CNN
+F 4 "71-CRCW0603-10K-E3" H 6900 4200 60  0001 C CNN "Mouse PN"
+	1    6900 4200
 	0    -1   -1   0
 $EndComp
@@
 $EndComp
 $Comp
-L CONN_01X01 P?
+L CONN_01X01 P20
 U 1 1 5609B537
 P 10500 2900
-F 0 "P?" H 10500 3000 50  0000 C CNN
+F 0 "P20" H 10500 3000 50  0000 C CNN
 F 1 "Jumper 1" H 10500 2800 50  0000 C CNN
 F 2 "Mounting_Holes:MountingHole_3mm" H 10500 2900 60  0001 C CNN
@@
 $EndComp
 $Comp
-L CONN_01X01 P?
+L CONN_01X01 P21
 U 1 1 5609B8CA
 P 10950 2900
-F 0 "P?" H 10950 3000 50  0000 C CNN
+F 0 "P21" H 10950 3000 50  0000 C CNN
 F 1 "Jumper 2" H 10950 2800 50  0000 C CNN
 F 2 "Mounting_Holes:MountingHole_3mm" H 10950 2900 60  0001 C CNN
@@
 $EndComp
 $Comp
-L CONN_01X01 P?
+L CONN_01X01 P23
 U 1 1 5609B9F5
 P 10500 3150
-F 0 "P?" H 10500 3250 50  0000 C CNN
+F 0 "P23" H 10500 3250 50  0000 C CNN
 F 1 "Jumper 3" H 10500 3050 50  0000 C CNN
 F 2 "Mounting_Holes:MountingHole_3mm" H 10500 3150 60  0001 C CNN
@@
 $EndComp
 $Comp
-L CONN_01X01 P?
+L CONN_01X01 P24
 U 1 1 5609B9FC
 P 10950 3150
-F 0 "P?" H 10950 3250 50  0000 C CNN
+F 0 "P24" H 10950 3250 50  0000 C CNN
 F 1 "Jumper 4" H 10950 3050 50  0000 C CNN
 F 2 "Mounting_Holes:MountingHole_3mm" H 10950 3150 60  0001 C CNN

Commit message: Split V2X in 2 boards, layout of SIM pcb done
Parts:
- removed R84, R86: DNS, Resistors_SMD:R_0603, symbol R
- removed R85: 0, Resistors_SMD:R_0603, symbol R
- added C68: 1U, Custom Parts:C_0603_SM, symbol C
- added C69: 100N, Custom Parts:C_0603_SM, symbol C
- added D18, D19: 4148, Custom Parts:Diode_0805_12_SM, symbol D
- added D20: GREEN, LEDs:LED-0805, symbol LED
- added Q19: 2N7000, Housings_SOT-23_SOT-143_TSOT-6:SOT-23, symbol Q_NMOS_SGD
- added R94: 22.1, Custom Parts:R_0603_sm, symbol R
- added R95: 330, Custom Parts:R_0603_sm, symbol R
- added R96: 47K, Custom Parts:R_0603_sm, symbol R
- C59, C60, C61, C62, C63: footprint Capacitors_SMD:C_0603 -> Custom Parts:C_0603_SM
- C64: footprint (none) -> Custom Parts:C_0603_SM
- CON1: footprint AVR-PDI-6 -> Pin_Headers:Pin_Header_Straight_2x03; symbol AVR-PDI-6 -> AVR-PDI-6-RESCUE-V2X
- FB6: footprint Capacitors_SMD:C_0805 -> Custom Parts:R_0603_sm
- IC1: footprint TQFP44 -> Housings_QFP:TQFP-44_10x10mm_Pitch0.8mm
- P20, P21, P23, P24: footprint Mounting_Holes:MountingHole_3mm -> Fiducials:Fiducial_1mm_Dia_2.54mm_Outer_CopperTop
- P22: footprint (none) -> Pin_Headers:Pin_Header_Straight_2x04
- Q16, Q17, Q18: footprint (none) -> Housings_SOT-23_SOT-143_TSOT-6:SOT-23
- R87, R88, R89, R90, R91, R92, R93: footprint Resistors_SMD:R_0603 -> Custom Parts:R_0603_sm
- U21: footprint (none) -> Housings_SOIC:SOIC-14_3.9x8.7mm_Pitch1.27mm
- U22, U23: footprint (none) -> Housings_SOIC:SOIC-16_3.9x9.9mm_Pitch1.27mm
Connections:
- net labels added: 3V3_E, BUTTON, PC_LED3, SEQ-CHGPUMP, SEQ_LED3
- net labels removed: 5V0_A, PC_RESET, SEQ_BUTTON, SEQ_WAKE, SIM_DTR, SIM_RI
- wire segments 42 -> 38
- no-connect marks 6 -> 3
Other:
- note added: "HUB Serial Data I2C/SMB\nHUB Serial Clock I2C/SMB\nACL Stream RXD to FTDI\nACL Stream TXD to FTDI"
- note added: "Host Power Short Circuit detect\nSEQ LED3 Output\nCAN Ctrl RXD from SEQ\nCAN Ctrl RXD from FTDI"
- note added: "Power-On expected negative pulse becomes \na SR positive pulse so default SR default 0 \nstate doesn't false start the SIM module."
- note added: "SEQ LED1 PWM Output\nSEQ LED2 PWM Output\nSIM TXD to SEQ\nSIM RXD to SEQ\nCHARGE PUMP SW\nButton (pwr/soft) input\nSEQ RXD to FTDI\nSEQ TXD to FTDI"
- note added: "SR clear outputs\nSR latch serial data \nCAN TXD to SEQ and FTDI\nCAN RXD to SEQ Buffer\nACL SPI Chip Select\nSR and ACL SPI Data OUT\nACL SPI Data IN\nSR and ACL Clock"
- note removed: "HUB Serial Data I2C/SMB\nHUB Serial Clock I2C/SMB\nAccel Stream RXD to FTDI\nAccel Stream TXD to FTDI"
- note removed: "Host Power Short Circuit detect\n\nCAN Ctrl RXD from PWRSEQ\nCAN Ctrl RXD from FTDI"
- note removed: "Power-On" negative pulse -> a SR positive pulse\nSo default SR state doesn't false start SIM module"
- note removed: "SEQ LED1 PWM Output\nSEQ LED2 PWM Output\nSIM TXD to PWRSEQ and FTDI\nSIM RXD to PWRSEQ Buffer\n\nButton (pwr/soft) input\nSEQ RXD to FTDI\nSEQ TXD to FTDI"
- note removed: "Shift Register clear outputs\nShift Register latch serial data \nCAN TXD to PWRSEQ and FTDI\nCAN RXD to PWRSEQ Buffer\nAccelerometer SPI Chip Select\nShift Register Data and SPI Data OUT\nAccelerometer SPI Data IN\nShift Register and Acceleromter Clock"
- moved on the sheet: D16, D17, Q17, Q18, R90, R91, R92, R93
