File: Hardware/Make Files/Active/V2X_CTRL.sch (KiCad schematic (older format))
At the start: 40 parts, among them CON1 AVR-PDI-6, IC1 ATXMEGA16A4U-A, P20 Jumper 1, P21 Jumper 2, P22 CONN_02X04, P23 Jumper 3, P24 Jumper 4, Q16 2N7000, Q17 2N7000, Q18 2N7000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

Commit message: work from home day
Parts:
- renumbered R19 to R18, R18 to R19
Connections:
- net 5V0_HOST: now also R19.2; no longer R18.1
- net HUB_ENABLE: now also R18.1; no longer R19.2
Other:
- moved on the sheet: R18, R19
Changed lines of the file:
@@
 HUB_ENABLE
 $Comp
-L R R18
+L R R19
 U 1 1 5621FEA5
-P 1650 700
-F 0 "R18" V 1730 700 50  0000 C CNN
-F 1 "0" V 1650 700 50  0000 C CNN
-F 2 "Custom Parts:R_0603_sm" V 1580 700 30  0001 C CNN
-F 3 "http://www.mouser.com/ds/2/427/dcrcwe3-109170.pdf" H 1650 700 30  0001 C CNN
-F 4 "71-CRCW0603-0-E3" H 1650 700 60  0001 C CNN "Mouse PN"
-	1    1650 700
+P 1650 900
+F 0 "R19" V 1730 900 50  0000 C CNN
+F 1 "0" V 1650 900 50  0000 C CNN
+F 2 "Custom Parts:R_0603_sm" V 1580 900 30  0001 C CNN
+F 3 "http://www.mouser.com/ds/2/427/dcrcwe3-109170.pdf" H 1650 900 30  0001 C CNN
+F 4 "71-CRCW0603-0-E3" H 1650 900 60  0001 C CNN "Mouse PN"
+	1    1650 900
 	0    1    -1   0
 $EndComp
 $Comp
-L R R19
+L R R18
 U 1 1 5622060B
-P 1650 900
-F 0 "R19" V 1730 900 50  0000 C CNN
-F 1 "DNS" V 1650 900 50  0000 C CNN
-F 2 "Custom Parts:R_0603_sm" V 1580 900 30  0001 C CNN
-F 3 "" H 1650 900 30  0000 C CNN
-	1    1650 900
+P 1650 700
+F 0 "R18" V 1730 700 50  0000 C CNN
+F 1 "DNS" V 1650 700 50  0000 C CNN
+F 2 "Custom Parts:R_0603_sm" V 1580 700 30  0001 C CNN
+F 3 "" H 1650 700 30  0000 C CNN
+	1    1650 700
 	0    -1   -1   0
 $EndComp

Commit message: home to work push
Parts:
- removed R18: DNS, Custom Parts:R_0603_sm, symbol R
- removed R19: 0, Custom Parts:R_0603_sm, symbol R
- removed R88, R89: 47K, Custom Parts:R_0603_sm, symbol R
- added R63: 1K, Custom Parts:R_0603_sm, symbol R
Connections:
- net CAN_RXD: now also R63.2; no longer U21.3
- new net: R63.1, U21.3
Other:
- note removed: "Determines ~RESET~ control for HUB"
- note removed: "Short Circuit Detection\n5V0_B_OUT is post poly fuse\nSample using logic level (maybe A2D)\nLogic '0' signal (<1.5V) indicates poly\nfuse is set, host output is in protect.\nLogic '1' signal (approx 2.4V) indicates\npoly fuse is clear, normal opperation.\nAn A2D value that is too high might \nindicate the Host is not attached."
Changed lines of the file:
@@
 SEQ_LED2
 $Comp
-L GND #PWR091
+L GND #PWR96
 U 1 1 55F86E9C
 P 4100 3900
-F 0 "#PWR091" H 4100 3650 50  0001 C CNN
+F 0 "#PWR96" H 4100 3650 50  0001 C CNN
 F 1 "GND" H 4100 3750 50  0000 C CNN
 F 2 "" H 4100 3900 60  0000 C CNN
@@
 	4350 1150 4350 1200
 Connection ~ 4250 1150
-Text GLabel 8900 5450 0    60   Input ~ 0
-5V0_B_OUT
-Wire Wire Line
-	8900 5450 8900 5550
-Wire Wire Line
-	8900 5850 8900 5950
-$Comp
-L GND #PWR092
-U 1 1 55F86EC1
-P 8900 6250
-F 0 "#PWR092" H 8900 6000 50  0001 C CNN
-F 1 "GND" H 8900 6100 50  0000 C CNN
-F 2 "" H 8900 6250 60  0000 C CNN
-F 3 "" H 8900 6250 60  0000 C CNN
-	1    8900 6250
-	1    0    0    -1
-$EndComp
-Text GLabel 8900 5900 0    60   Input ~ 0
-HOST_SC
 Text GLabel 5150 2450 2    60   Input ~ 0
 HOST_SC
-Text Notes 9150 6300 0    60   ~ 0
-Short Circuit Detection\n5V0_B_OUT is post poly fuse\nSample using logic level (maybe A2D)\nLogic '0' signal (<1.5V) indicates poly\nfuse is set, host output is in protect.\nLogic '1' signal (approx 2.4V) indicates\npoly fuse is clear, normal opperation.\nAn A2D value that is too high might \nindicate the Host is not attached.
 $Comp
 L ATXMEGA16A4U-A IC1
@@
 PDI
 $Comp
-L GND #PWR093
+L GND #PWR95
 U 1 1 55F86EF0
 P 2000 2050
-F 0 "#PWR093" H 2000 1800 50  0001 C CNN
+F 0 "#PWR95" H 2000 1800 50  0001 C CNN
 F 1 "GND" H 2000 1900 50  0000 C CNN
 F 2 "" H 2000 2050 60  0000 C CNN
@@
 Text GLabel 9100 2300 0    60   Input ~ 0
 CAN_RXD_FTDI
-Text GLabel 10000 1700 2    60   Input ~ 0
+Text GLabel 10300 1700 2    60   Input ~ 0
 CAN_RXD
 Text GLabel 10000 2300 2    60   Input ~ 0
@@
 5V0_B_EN
 $Comp
-L GND #PWR094
+L GND #PWR93
 U 1 1 55FA434A
 P 1100 5750
-F 0 "#PWR094" H 1100 5500 50  0001 C CNN
+F 0 "#PWR93" H 1100 5500 50  0001 C CNN
 F 1 "GND" H 1100 5600 50  0000 C CNN
 F 2 "" H 1100 5750 60  0000 C CNN
@@
 $EndComp
 $Comp
-L GND #PWR095
+L GND #PWR94
 U 1 1 55FA46C8
 P 1100 7150
-F 0 "#PWR095" H 1100 6900 50  0001 C CNN
+F 0 "#PWR94" H 1100 6900 50  0001 C CNN
 F 1 "GND" H 1100 7000 50  0000 C CNN
 F 2 "" H 1100 7150 60  0000 C CNN
@@
 $EndComp
 $Comp
-L GND #PWR096
+L GND #PWR100
 U 1 1 55FD726F
 P 5850 7350
-F 0 "#PWR096" H 5850 7100 50  0001 C CNN
+F 0 "#PWR100" H 5850 7100 50  0001 C CNN
 F 1 "GND" H 5850 7200 50  0000 C CNN
 F 2 "" H 5850 7350 60  0000 C CNN
@@
 $EndComp
 $Comp
-L GND #PWR097
+L GND #PWR99
 U 1 1 55FD7284
 P 5500 7500
-F 0 "#PWR097" H 5500 7250 50  0001 C CNN
+F 0 "#PWR99" H 5500 7250 50  0001 C CNN
 F 1 "GND" H 5500 7350 50  0000 C CNN
 F 2 "" H 5500 7500 60  0000 C CNN
@@
 $EndComp
 $Comp
-L GND #PWR098
+L GND #PWR101
 U 1 1 55FD7672
 P 6350 7500
-F 0 "#PWR098" H 6350 7250 50  0001 C CNN
+F 0 "#PWR101" H 6350 7250 50  0001 C CNN
 F 1 "GND" H 6350 7350 50  0000 C CNN
 F 2 "" H 6350 7500 60  0000 C CNN
@@
 	6350 7000 6350 7200
 $Comp
-L GND #PWR099
+L GND #PWR103
 U 1 1 55FD7660
 P 6700 7350
-F 0 "#PWR099" H 6700 7100 50  0001 C CNN
+F 0 "#PWR103" H 6700 7100 50  0001 C CNN
 F 1 "GND" H 6700 7200 50  0000 C CNN
 F 2 "" H 6700 7350 60  0000 C CNN
@@
 $EndComp
 $Comp
-L GND #PWR0100
+L GND #PWR102
 U 1 1 55FE1020
 P 6400 4850
-F 0 "#PWR0100" H 6400 4600 50  0001 C CNN
+F 0 "#PWR102" H 6400 4600 50  0001 C CNN
 F 1 "GND" H 6400 4700 50  0000 C CNN
 F 2 "" H 6400 4850 60  0000 C CNN
@@
 Connection ~ 10550 750
 $Comp
-L GND #PWR0101
+L GND #PWR111
 U 1 1 56006FBB
 P 10550 1100
-F 0 "#PWR0101" H 10550 850 50  0001 C CNN
+F 0 "#PWR111" H 10550 850 50  0001 C CNN
 F 1 "GND" H 10550 950 50  0000 C CNN
 F 2 "" H 10550 1100 60  0000 C CNN
@@
 Connection ~ 9000 750
 $Comp
-L GND #PWR0102
+L GND #PWR107
 U 1 1 560285A0
 P 9000 1100
-F 0 "#PWR0102" H 9000 850 50  0001 C CNN
+F 0 "#PWR107" H 9000 850 50  0001 C CNN
 F 1 "GND" H 9000 950 50  0000 C CNN
 F 2 "" H 9000 1100 60  0000 C CNN
@@
 $EndComp
 $Comp
-L GND #PWR0103
+L GND #PWR109
 U 1 1 560285F6
 P 9300 1100
-F 0 "#PWR0103" H 9300 850 50  0001 C CNN
+F 0 "#PWR109" H 9300 850 50  0001 C CNN
 F 1 "GND" H 9300 950 50  0000 C CNN
 F 2 "" H 9300 1100 60  0000 C CNN
@@
 $EndComp
 $Comp
-L GND #PWR0104
+L GND #PWR110
 U 1 1 5602864C
 P 9600 1100
-F 0 "#PWR0104" H 9600 850 50  0001 C CNN
+F 0 "#PWR110" H 9600 850 50  0001 C CNN
 F 1 "GND" H 9600 950 50  0000 C CNN
 F 2 "" H 9600 1100 60  0000 C CNN
@@
 Connection ~ 9150 750
 $Comp
-L VCC #PWR0105
+L VCC #PWR108
 U 1 1 56029609
 P 9150 700
-F 0 "#PWR0105" H 9150 550 50  0001 C CNN
+F 0 "#PWR108" H 9150 550 50  0001 C CNN
 F 1 "VCC" H 9150 850 50  0000 C CNN
 F 2 "" H 9150 700 60  0000 C CNN
@@
 Connection ~ 8750 750
 $Comp
-L GND #PWR0106
+L GND #PWR106
 U 1 1 5602C4DB
 P 8750 1100
-F 0 "#PWR0106" H 8750 850 50  0001 C CNN
+F 0 "#PWR106" H 8750 850 50  0001 C CNN
 F 1 "GND" H 8750 950 50  0000 C CNN
 F 2 "" H 8750 1100 60  0000 C CNN
@@
 $EndComp
 $Comp
-L GND #PWR0107
+L GND #PWR105
 U 1 1 5602C537
 P 8450 1100
-F 0 "#PWR0107" H 8450 850 50  0001 C CNN
+F 0 "#PWR105" H 8450 850 50  0001 C CNN
 F 1 "GND" H 8450 950 50  0000 C CNN
 F 2 "" H 8450 1100 60  0000 C CNN
@@
 $EndComp
 $Comp
-L R R89
-U 1 1 5605AB0D
-P 8900 6100
-F 0 "R89" V 8980 6100 50  0000 C CNN
-F 1 "47K" V 8900 6100 50  0000 C CNN
-F 2 "Custom Parts:R_0603_sm" V 8830 6100 30  0001 C CNN
-F 3 "http://www.mouser.com/ds/2/427/dcrcwe3-109170.pdf" H 8900 6100 30  0001 C CNN
-F 4 "71-CRCW0603-47K-E3" H 8900 6100 60  0001 C CNN "Mouse PN"
-	1    8900 6100
-	-1   0    0    1
-$EndComp
-$Comp
-L R R88
-U 1 1 5605AB9B
-P 8900 5700
-F 0 "R88" V 8980 5700 50  0000 C CNN
-F 1 "47K" V 8900 5700 50  0000 C CNN
-F 2 "Custom Parts:R_0603_sm" V 8830 5700 30  0001 C CNN
-F 3 "http://www.mouser.com/ds/2/427/dcrcwe3-109170.pdf" H 8900 5700 30  0001 C CNN
-F 4 "71-CRCW0603-47K-E3" H 8900 5700 60  0001 C CNN "Mouse PN"
-	1    8900 5700
-	-1   0    0    1
-$EndComp
-$Comp
 L R R87
 U 1 1 5605AFDD
@@
 $EndComp
 $Comp
-L GND #PWR0108
+L GND #PWR98
 U 1 1 560D95B8
 P 5000 7350
-F 0 "#PWR0108" H 5000 7100 50  0001 C CNN
+F 0 "#PWR98" H 5000 7100 50  0001 C CNN
 F 1 "GND" H 5000 7200 50  0000 C CNN
 F 2 "" H 5000 7350 60  0000 C CNN
@@
 $EndComp
 $Comp
-L GND #PWR0109
+L GND #PWR97
 U 1 1 560D95C5
 P 4650 7500
-F 0 "#PWR0109" H 4650 7250 50  0001 C CNN
+F 0 "#PWR97" H 4650 7250 50  0001 C CNN
 F 1 "GND" H 4650 7350 50  0000 C CNN
 F 2 "" H 4650 7500 60  0000 C CNN
@@
 $EndComp
 $Comp
-L GND #PWR0110
+L GND #PWR104
 U 1 1 560DBE9F
 P 7550 1150
-F 0 "#PWR0110" H 7550 900 50  0001 C CNN
+F 0 "#PWR104" H 7550 900 50  0001 C CNN
 F 1 "GND" H 7550 1000 50  0000 C CNN
 F 2 "" H 7550 1150 60  0000 C CNN
@@
 Text Notes 5550 900  0    69   ~ 0
 LED Charge pump. \nToggle pin state \nat approx 100khz
-Text GLabel 2000 700  2    60   Input ~ 0
-~HUB_RESET
-Text GLabel 1400 900  0    60   Input ~ 0
-5V0_HOST
-Text GLabel 1400 700  0    60   Input ~ 0
-HUB_ENABLE
-$Comp
-L R R19
-U 1 1 5621FEA5
-P 1650 900
-F 0 "R19" V 1730 900 50  0000 C CNN
-F 1 "0" V 1650 900 50  0000 C CNN
-F 2 "Custom Parts:R_0603_sm" V 1580 900 30  0001 C CNN
-F 3 "http://www.mouser.com/ds/2/427/dcrcwe3-109170.pdf" H 1650 900 30  0001 C CNN
-F 4 "71-CRCW0603-0-E3" H 1650 900 60  0001 C CNN "Mouse PN"
-	1    1650 900
-	0    1    -1   0
-$EndComp
-$Comp
-L R R18
-U 1 1 5622060B
-P 1650 700
-F 0 "R18" V 1730 700 50  0000 C CNN
-F 1 "DNS" V 1650 700 50  0000 C CNN
-F 2 "Custom Parts:R_0603_sm" V 1580 700 30  0001 C CNN
-F 3 "" H 1650 700 30  0000 C CNN
-	1    1650 700
+Wire Notes Line
+	500  1200 3450 1200
+Wire Notes Line
+	500  2250 2850 2250
+Wire Notes Line
+	2850 2250 2850 1900
+Wire Notes Line
+	2850 1900 3450 1900
+Wire Notes Line
+	3450 1900 3450 1200
+$Comp
+L R R63
+U 1 1 56280EFC
+P 10150 1700
+F 0 "R63" V 10230 1700 50  0000 C CNN
+F 1 "1K" V 10150 1700 50  0000 C CNN
+F 2 "Custom Parts:R_0603_sm" V 10080 1700 30  0001 C CNN
+F 3 "http://www.mouser.com/ds/2/427/dcrcwe3-109170.pdf" H 10150 1700 30  0001 C CNN
+F 4 "71-CRCW0603-1.0K-E3" H 10150 1700 60  0001 C CNN "Mouse PN"
+	1    10150 1700
 	0    -1   -1   0
 $EndComp
-Wire Wire Line
-	1800 700  2000 700
-Wire Wire Line
-	1900 700  1900 900
-Wire Wire Line
-	1900 900  1800 900
-Connection ~ 1900 700
-Wire Wire Line
-	1500 700  1400 700
-Wire Wire Line
-	1400 900  1500 900
-Text Notes 700  1100 0    69   ~ 0
-Determines ~RESET~ control for HUB
-Wire Notes Line
-	2750 500  2750 1200
-Wire Notes Line
-	500  1200 3450 1200
-Wire Notes Line
-	500  2250 2850 2250
-Wire Notes Line
-	2850 2250 2850 1900
-Wire Notes Line
-	2850 1900 3450 1900
-Wire Notes Line
-	3450 1900 3450 1200
 $EndSCHEMATC
