File: Hardware/Make Files/Active/_saved_V2X_HUB.sch (KiCad schematic (older format))
At the start: 13 parts, among them U20 USB2242, X3 24MHz

Commit message: work from home day
Parts:
- added R18: DNS, Custom Parts:R_0603_sm, symbol R
- added R19, R60: 47K, Custom Parts:R_0603_sm, symbol R
Connections:
- net GND: now also R60.2
- net ~HUB_RESET: now also R18.2, R19.2, R60.1
- new net 5V0_HOST: R19.1
- new net HUB_ENABLE: R18.1
Other:
- note added: "Determines ~RESET~ control for HUB\nSet to Auto Host 5V0 detect"
- moved on the sheet: R81, R82, R83, X3
Changed lines of the file:
@@
 3V3_B
 $Comp
-L GND #PWR082
+L GND #PWR86
 U 1 1 55F890DF
 P 3450 2300
-F 0 "#PWR082" H 3450 2050 50  0001 C CNN
+F 0 "#PWR86" H 3450 2050 50  0001 C CNN
 F 1 "GND" V 3450 2100 50  0000 C CNN
 F 2 "" H 3450 2300 60  0000 C CNN
@@
 Text GLabel 4150 1250 2    60   Input ~ 0
 HUB_CLKN
-Text GLabel 3350 6450 2    60   Input ~ 0
+Text GLabel 6200 7150 2    60   Input ~ 0
 HUB_CLK
-Text GLabel 2650 6450 0    60   Input ~ 0
+Text GLabel 5500 7150 0    60   Input ~ 0
 HUB_CLKN
 Wire Wire Line
-	2650 6450 2800 6450
-Wire Wire Line
-	3200 6450 3350 6450
-$Comp
-L GND #PWR083
+	5500 7150 5650 7150
+Wire Wire Line
+	6050 7150 6200 7150
+$Comp
+L GND #PWR85
 U 1 1 55F89454
-P 3000 6550
-F 0 "#PWR083" H 3000 6300 50  0001 C CNN
-F 1 "GND" V 3000 6350 50  0000 C CNN
-F 2 "" H 3000 6550 60  0000 C CNN
-F 3 "" H 3000 6550 60  0000 C CNN
-	1    3000 6550
+P 5850 7250
+F 0 "#PWR85" H 5850 7000 50  0001 C CNN
+F 1 "GND" V 5850 7050 50  0000 C CNN
+F 2 "" H 5850 7250 60  0000 C CNN
+F 3 "" H 5850 7250 60  0000 C CNN
+	1    5850 7250
 	1    0    0    -1
 $EndComp
@@
 L R R81
 U 1 1 55F8A6E8
-P 3750 5100
-F 0 "R81" V 3830 5100 50  0000 C CNN
-F 1 "DNS" V 3750 5100 50  0000 C CNN
-F 2 "Custom Parts:R_0603_sm" V 3680 5100 30  0001 C CNN
-F 3 "" H 3750 5100 30  0000 C CNN
-	1    3750 5100
+P 7300 3450
+F 0 "R81" V 7380 3450 50  0000 C CNN
+F 1 "DNS" V 7300 3450 50  0000 C CNN
+F 2 "Custom Parts:R_0603_sm" V 7230 3450 30  0001 C CNN
+F 3 "" H 7300 3450 30  0000 C CNN
+	1    7300 3450
 	-1   0    0    1
 $EndComp
@@
 L R R83
 U 1 1 55F8A750
-P 3750 5600
-F 0 "R83" V 3830 5600 50  0000 C CNN
-F 1 "1K0" V 3750 5600 50  0000 C CNN
-F 2 "Custom Parts:R_0603_sm" V 3680 5600 30  0001 C CNN
-F 3 "http://www.vishay.com/doc?20035" H 3750 5600 30  0001 C CNN
-F 4 "71-CRCW0603-1.0K-E3" H 3750 5600 60  0001 C CNN "Mouse PN"
-	1    3750 5600
+P 7300 3950
+F 0 "R83" V 7380 3950 50  0000 C CNN
+F 1 "1K0" V 7300 3950 50  0000 C CNN
+F 2 "Custom Parts:R_0603_sm" V 7230 3950 30  0001 C CNN
+F 3 "http://www.vishay.com/doc?20035" H 7300 3950 30  0001 C CNN
+F 4 "71-CRCW0603-1.0K-E3" H 7300 3950 60  0001 C CNN "Mouse PN"
+	1    7300 3950
 	-1   0    0    1
 $EndComp
 Wire Wire Line
-	3750 5250 3750 5450
-Connection ~ 3750 5350
-Text GLabel 3650 4850 0    60   Input ~ 0
+	7300 3600 7300 3800
+Connection ~ 7300 3700
+Text GLabel 7200 3200 0    60   Input ~ 0
 3V3_B
 $Comp
-L GND #PWR084
+L GND #PWR88
 U 1 1 55F8A8AD
-P 3750 5750
-F 0 "#PWR084" H 3750 5500 50  0001 C CNN
-F 1 "GND" V 3750 5550 50  0000 C CNN
-F 2 "" H 3750 5750 60  0000 C CNN
-F 3 "" H 3750 5750 60  0000 C CNN
-	1    3750 5750
-	1    0    0    -1
-$EndComp
-Wire Wire Line
-	3750 4950 3750 4850
-Wire Wire Line
-	3750 4850 3650 4850
-Text Notes 1900 5300 0    60   ~ 0
+P 7300 4100
+F 0 "#PWR88" H 7300 3850 50  0001 C CNN
+F 1 "GND" V 7300 3900 50  0000 C CNN
+F 2 "" H 7300 4100 60  0000 C CNN
+F 3 "" H 7300 4100 60  0000 C CNN
+	1    7300 4100
+	1    0    0    -1
+$EndComp
+Wire Wire Line
+	7300 3300 7300 3200
+Wire Wire Line
+	7300 3200 7200 3200
+Text Notes 5450 3650 0    60   ~ 0
 Boot Strapping Option\nPRTPWR1 = Battery Charge Enable\n0  = feature off, we dont need.
 $Comp
-L GND #PWR085
+L GND #PWR90
 U 1 1 55F8AB65
 P 5100 950
-F 0 "#PWR085" H 5100 700 50  0001 C CNN
+F 0 "#PWR90" H 5100 700 50  0001 C CNN
 F 1 "GND" V 5100 750 50  0000 C CNN
 F 2 "" H 5100 950 60  0000 C CNN
@@
 Connection ~ 1250 1750
 $Comp
-L GND #PWR086
+L GND #PWR82
 U 1 1 55F8AFDA
 P 1250 2050
-F 0 "#PWR086" H 1250 1800 50  0001 C CNN
+F 0 "#PWR82" H 1250 1800 50  0001 C CNN
 F 1 "GND" V 1250 1850 50  0000 C CNN
 F 2 "" H 1250 2050 60  0000 C CNN
@@
 Connection ~ 1750 950
 $Comp
-L GND #PWR087
+L GND #PWR84
 U 1 1 55F8B30B
 P 1750 1250
-F 0 "#PWR087" H 1750 1000 50  0001 C CNN
+F 0 "#PWR84" H 1750 1000 50  0001 C CNN
 F 1 "GND" V 1750 1050 50  0000 C CNN
 F 2 "" H 1750 1250 60  0000 C CNN
@@
 	1600 1850 2750 1850
 $Comp
-L GND #PWR088
+L GND #PWR83
 U 1 1 55F8B452
 P 1600 2300
-F 0 "#PWR088" H 1600 2050 50  0001 C CNN
+F 0 "#PWR83" H 1600 2050 50  0001 C CNN
 F 1 "GND" V 1600 2100 50  0000 C CNN
 F 2 "" H 1600 2300 60  0000 C CNN
@@
 	4150 1050 4800 1050
 $Comp
-L GND #PWR089
+L GND #PWR89
 U 1 1 55F8B6A0
 P 4800 1350
-F 0 "#PWR089" H 4800 1100 50  0001 C CNN
+F 0 "#PWR89" H 4800 1100 50  0001 C CNN
 F 1 "GND" V 4800 1150 50  0000 C CNN
 F 2 "" H 4800 1350 60  0000 C CNN
@@
 	1    0    0    -1
 $EndComp
-Text Notes 1950 5700 0    60   ~ 0
+Text Notes 5500 4050 0    60   ~ 0
 PRTPWR1 and PRTPWR2 go\n high when the port is active
 Text GLabel 4150 1750 2    60   Input ~ 0
 3V3_B
 Wire Wire Line
-	3650 5400 3750 5400
-Connection ~ 3750 5400
+	7200 3750 7300 3750
+Connection ~ 7300 3750
 Text GLabel 4150 1950 2    60   Input ~ 0
 HUB_SCL
@@
 HUB_SDA
 $Comp
-L GND #PWR090
+L GND #PWR87
 U 1 1 55F9C2E3
 P 3700 4250
-F 0 "#PWR090" H 3700 4000 50  0001 C CNN
+F 0 "#PWR87" H 3700 4000 50  0001 C CNN
 F 1 "GND" V 3700 4050 50  0000 C CNN
 F 2 "" H 3700 4250 60  0000 C CNN
@@
 Text GLabel 2750 1550 0    69   Input ~ 0
 HUB_PWR_PRT1
-Text GLabel 4150 5350 2    69   Input ~ 0
+Text GLabel 7700 3700 2    69   Input ~ 0
 HUB_STATUS
 Text GLabel 4150 3850 2    69   Input ~ 0
@@
 Wire Wire Line
 	3850 3850 3700 3850
-Text GLabel 3650 5400 0    69   Input ~ 0
+Text GLabel 7200 3750 0    69   Input ~ 0
 HUB_PWR_PRT1
 Wire Wire Line
-	3750 5350 3850 5350
+	7300 3700 7400 3700
 Text GLabel 4150 1550 2    60   Input ~ 0
 3V3_B
@@
 L R R82
 U 1 1 56070A80
-P 4000 5350
-F 0 "R82" V 4080 5350 50  0000 C CNN
-F 1 "1K0" V 4000 5350 50  0000 C CNN
-F 2 "Custom Parts:R_0603_sm" V 3930 5350 30  0001 C CNN
-F 3 "http://www.vishay.com/doc?20035" H 4000 5350 30  0001 C CNN
-F 4 "71-CRCW0603-1.0K-E3" H 4000 5350 60  0001 C CNN "Mouse PN"
-	1    4000 5350
+P 7550 3700
+F 0 "R82" V 7630 3700 50  0000 C CNN
+F 1 "1K0" V 7550 3700 50  0000 C CNN
+F 2 "Custom Parts:R_0603_sm" V 7480 3700 30  0001 C CNN
+F 3 "http://www.vishay.com/doc?20035" H 7550 3700 30  0001 C CNN
+F 4 "71-CRCW0603-1.0K-E3" H 7550 3700 60  0001 C CNN "Mouse PN"
+	1    7550 3700
 	0    -1   -1   0
 $EndComp
@@
 L CRYSTAL_SMD X3
 U 1 1 56092E15
-P 3000 6450
-F 0 "X3" H 3000 6540 50  0000 C CNN
-F 1 "24MHz" H 3030 6340 50  0000 L CNN
-F 2 "Custom Parts:AWSCR" H 3000 6450 60  0001 C CNN
-F 3 "http://www.abracon.com/Resonators/N_AWSCR-MT.pdf" H 3000 6450 60  0001 C CNN
-F 4 "815-AWSCR-24.00MTD-T" H 3000 6450 60  0001 C CNN "Mouse PN"
-	1    3000 6450
-	1    0    0    -1
+P 5850 7150
+F 0 "X3" H 5850 7240 50  0000 C CNN
+F 1 "24MHz" H 5880 7040 50  0000 L CNN
+F 2 "Custom Parts:AWSCR" H 5850 7150 60  0001 C CNN
+F 3 "http://www.abracon.com/Resonators/N_AWSCR-MT.pdf" H 5850 7150 60  0001 C CNN
+F 4 "815-AWSCR-24.00MTD-T" H 5850 7150 60  0001 C CNN "Mouse PN"
+	1    5850 7150
+	1    0    0    -1
+$EndComp
+Text GLabel 7500 1000 2    60   Input ~ 0
+~HUB_RESET
+Text GLabel 6900 1200 0    60   Input ~ 0
+5V0_HOST
+Text GLabel 6900 1000 0    60   Input ~ 0
+HUB_ENABLE
+$Comp
+L R R18
+U 1 1 5627870C
+P 7150 1000
+F 0 "R18" V 7230 1000 50  0000 C CNN
+F 1 "DNS" V 7150 1000 50  0000 C CNN
+F 2 "Custom Parts:R_0603_sm" V 7080 1000 30  0001 C CNN
+F 3 "" H 7150 1000 30  0000 C CNN
+	1    7150 1000
+	0    -1   -1   0
+$EndComp
+Wire Wire Line
+	7300 1000 7500 1000
+Wire Wire Line
+	7400 1000 7400 1200
+Wire Wire Line
+	7300 1200 7500 1200
+Connection ~ 7400 1000
+Wire Wire Line
+	7000 1000 6900 1000
+Wire Wire Line
+	6900 1200 7000 1200
+Text Notes 6200 1500 0    69   ~ 0
+Determines ~RESET~ control for HUB\nSet to Auto Host 5V0 detect
+$Comp
+L R R19
+U 1 1 5627871B
+P 7150 1200
+F 0 "R19" V 7230 1200 50  0000 C CNN
+F 1 "47K" V 7150 1200 50  0000 C CNN
+F 2 "Custom Parts:R_0603_sm" V 7080 1200 30  0001 C CNN
+F 3 "http://www.mouser.com/ds/2/427/dcrcwe3-109170.pdf" H 7150 1200 30  0001 C CNN
+F 4 "71-CRCW0603-47K-E3" H 7150 1200 60  0001 C CNN "Mouse PN"
+	1    7150 1200
+	0    -1   -1   0
+$EndComp
+$Comp
+L R R60
+U 1 1 56278723
+P 7650 1200
+F 0 "R60" V 7730 1200 50  0000 C CNN
+F 1 "47K" V 7650 1200 50  0000 C CNN
+F 2 "Custom Parts:R_0603_sm" V 7580 1200 30  0001 C CNN
+F 3 "http://www.mouser.com/ds/2/427/dcrcwe3-109170.pdf" H 7650 1200 30  0001 C CNN
+F 4 "71-CRCW0603-47K-E3" H 7650 1200 60  0001 C CNN "Mouse PN"
+	1    7650 1200
+	0    -1   -1   0
+$EndComp
+Connection ~ 7400 1200
+$Comp
+L GND #PWR91
+U 1 1 5627872B
+P 7800 1200
+F 0 "#PWR91" H 7800 950 50  0001 C CNN
+F 1 "GND" V 7800 1000 50  0000 C CNN
+F 2 "" H 7800 1200 60  0000 C CNN
+F 3 "" H 7800 1200 60  0000 C CNN
+	1    7800 1200
+	0    -1   -1   0
 $EndComp
 $EndSCHEMATC
