File: Hardware/Make Files/Active/_saved_V2X_PWR.sch (KiCad schematic (older format))
At the start: 58 parts, among them P10 Board Mount 2, P11 Ficudial2, P12 Board Mount 3, P13 Ficudial3, P15 Board Mount 4, P16 Ficudial4, P17 CUR_SEN, P19 CUR_SEN, P6 Board Mount 1, P7 Ficudial1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

Commit message: work from home day
Parts:
- added R88, R89: 47K, Custom Parts:R_0603_sm, symbol R
- gave numbers to parts that had none: 3
Connections:
- net 5V0_B_OUT: now also R88.2
- net GND: now also R89.1
- new net HOST_SC: R88.1, R89.2
Other:
- note added: "Short Circuit Detection\n5V0_B_OUT is post poly fuse\nSample using logic level (maybe A2D)\nLogic '0' signal (<1.5V) indicates poly\nfuse is set, host output is in protect.\nLogic '1' signal (approx 2.4V) indicates\npoly fuse is clear, normal opperation.\nAn A2D value that is too high might \nindicate the Host is not attached."
Changed lines of the file:
@@
 Connection ~ 2900 1050
 $Comp
-L GND #PWR051
+L GND #PWR54
 U 1 1 55AAAD3C
 P 1700 1400
-F 0 "#PWR051" H 1700 1150 50  0001 C CNN
+F 0 "#PWR54" H 1700 1150 50  0001 C CNN
 F 1 "GND" H 1700 1250 50  0000 C CNN
 F 2 "" H 1700 1400 60  0000 C CNN
@@
 $EndComp
 $Comp
-L GND #PWR052
+L GND #PWR58
 U 1 1 55AAAECD
 P 2400 1500
-F 0 "#PWR052" H 2400 1250 50  0001 C CNN
+F 0 "#PWR58" H 2400 1250 50  0001 C CNN
 F 1 "GND" H 2400 1350 50  0000 C CNN
 F 2 "" H 2400 1500 60  0000 C CNN
@@
 $EndComp
 $Comp
-L GND #PWR053
+L GND #PWR62
 U 1 1 55AAAF11
 P 2900 1450
-F 0 "#PWR053" H 2900 1200 50  0001 C CNN
+F 0 "#PWR62" H 2900 1200 50  0001 C CNN
 F 1 "GND" H 2900 1300 50  0000 C CNN
 F 2 "" H 2900 1450 60  0000 C CNN
@@
 3.3V @ 1A DC-DC Power Supply
 $Comp
-L GND #PWR054
+L GND #PWR72
 U 1 1 55C7D0D4
 P 7700 2900
-F 0 "#PWR054" H 7700 2650 50  0001 C CNN
+F 0 "#PWR72" H 7700 2650 50  0001 C CNN
 F 1 "GND" H 7700 2750 50  0000 C CNN
 F 2 "" H 7700 2900 60  0000 C CNN
@@
 $EndComp
 $Comp
-L GND #PWR055
+L GND #PWR52
 U 1 1 55FBBA0A
 P 1350 2400
-F 0 "#PWR055" H 1350 2150 50  0001 C CNN
+F 0 "#PWR52" H 1350 2150 50  0001 C CNN
 F 1 "GND" V 1350 2200 50  0000 C CNN
 F 2 "" H 1350 2400 60  0000 C CNN
@@
 $EndComp
 $Comp
-L GND #PWR056
+L GND #PWR65
 U 1 1 55FBBA10
 P 3450 3100
-F 0 "#PWR056" H 3450 2850 50  0001 C CNN
+F 0 "#PWR65" H 3450 2850 50  0001 C CNN
 F 1 "GND" H 3450 2950 50  0000 C CNN
 F 2 "" H 3450 3100 60  0000 C CNN
@@
 Connection ~ 2800 2300
 $Comp
-L GND #PWR057
+L GND #PWR61
 U 1 1 55FBBA33
 P 2800 2600
-F 0 "#PWR057" H 2800 2350 50  0001 C CNN
+F 0 "#PWR61" H 2800 2350 50  0001 C CNN
 F 1 "GND" H 2950 2550 50  0000 C CNN
 F 2 "" H 2800 2600 60  0000 C CNN
@@
 $EndComp
 $Comp
-L GND #PWR058
+L GND #PWR57
 U 1 1 55FBBA3F
 P 2250 2800
-F 0 "#PWR058" H 2250 2550 50  0001 C CNN
+F 0 "#PWR57" H 2250 2550 50  0001 C CNN
 F 1 "GND" V 2250 2600 50  0000 C CNN
 F 2 "" H 2250 2800 60  0000 C CNN
@@
 Connection ~ 1300 2800
 $Comp
-L GND #PWR059
+L GND #PWR51
 U 1 1 55FBBA68
 P 950 2800
-F 0 "#PWR059" H 950 2550 50  0001 C CNN
+F 0 "#PWR51" H 950 2550 50  0001 C CNN
 F 1 "GND" V 950 2600 50  0000 C CNN
 F 2 "" H 950 2800 60  0000 C CNN
@@
 5V0_A
 $Comp
-L GND #PWR060
+L GND #PWR66
 U 1 1 55FBD5DC
 P 3450 4050
-F 0 "#PWR060" H 3450 3800 50  0001 C CNN
+F 0 "#PWR66" H 3450 3800 50  0001 C CNN
 F 1 "GND" V 3450 3850 50  0000 C CNN
 F 2 "" H 3450 4050 60  0000 C CNN
@@
 $EndComp
 $Comp
-L GND #PWR061
+L GND #PWR70
 U 1 1 55FBD5E2
 P 5550 4750
-F 0 "#PWR061" H 5550 4500 50  0001 C CNN
+F 0 "#PWR70" H 5550 4500 50  0001 C CNN
 F 1 "GND" H 5550 4600 50  0000 C CNN
 F 2 "" H 5550 4750 60  0000 C CNN
@@
 $EndComp
 $Comp
-L GND #PWR062
+L GND #PWR69
 U 1 1 55FBD605
 P 4900 4250
-F 0 "#PWR062" H 4900 4000 50  0001 C CNN
+F 0 "#PWR69" H 4900 4000 50  0001 C CNN
 F 1 "GND" H 5050 4200 50  0000 C CNN
 F 2 "" H 4900 4250 60  0000 C CNN
@@
 $EndComp
 $Comp
-L GND #PWR063
+L GND #PWR68
 U 1 1 55FBD611
 P 4350 4450
-F 0 "#PWR063" H 4350 4200 50  0001 C CNN
+F 0 "#PWR68" H 4350 4200 50  0001 C CNN
 F 1 "GND" V 4350 4250 50  0000 C CNN
 F 2 "" H 4350 4450 60  0000 C CNN
@@
 	3400 4150 3450 4150
 $Comp
-L GND #PWR064
+L GND #PWR67
 U 1 1 55FBD63A
 P 3450 5050
-F 0 "#PWR064" H 3450 4800 50  0001 C CNN
+F 0 "#PWR67" H 3450 4800 50  0001 C CNN
 F 1 "GND" V 3450 4850 50  0000 C CNN
 F 2 "" H 3450 5050 60  0000 C CNN
@@
 5V0_B_EN
 $Comp
-L GND #PWR065
+L GND #PWR71
 U 1 1 55FC949A
 P 5900 2700
-F 0 "#PWR065" H 5900 2450 50  0001 C CNN
+F 0 "#PWR71" H 5900 2450 50  0001 C CNN
 F 1 "GND" H 5900 2550 50  0000 C CNN
 F 2 "" H 5900 2700 60  0000 C CNN
@@
 $EndComp
 $Comp
-L GND #PWR066
+L GND #PWR53
 U 1 1 55FCD01A
 P 1350 4750
-F 0 "#PWR066" H 1350 4500 50  0001 C CNN
+F 0 "#PWR53" H 1350 4500 50  0001 C CNN
 F 1 "GND" V 1450 4700 50  0000 C CNN
 F 2 "" H 1350 4750 60  0000 C CNN
@@
 $EndComp
 $Comp
-L GND #PWR067
+L GND #PWR73
 U 1 1 55FCEBFC
 P 7800 4000
-F 0 "#PWR067" H 7800 3750 50  0001 C CNN
+F 0 "#PWR73" H 7800 3750 50  0001 C CNN
 F 1 "GND" H 7800 3850 50  0000 C CNN
 F 2 "" H 7800 4000 60  0000 C CNN
@@
 $EndComp
 $Comp
-L GND #PWR068
+L GND #PWR56
 U 1 1 5600FC76
 P 2000 4300
-F 0 "#PWR068" H 2000 4050 50  0001 C CNN
+F 0 "#PWR56" H 2000 4050 50  0001 C CNN
 F 1 "GND" V 2100 4250 50  0000 C CNN
 F 2 "" H 2000 4300 60  0000 C CNN
@@
 	1700 4550 1700 4600
 $Comp
-L GND #PWR069
+L GND #PWR55
 U 1 1 56011CFE
 P 1700 4900
-F 0 "#PWR069" H 1700 4650 50  0001 C CNN
+F 0 "#PWR55" H 1700 4650 50  0001 C CNN
 F 1 "GND" H 1700 4750 50  0000 C CNN
 F 2 "" H 1700 4900 60  0000 C CNN
@@
 Text Notes 4500 2950 0    69   ~ 0
 Slew Rate is\nControlable
-Text Notes 6500 4250 0    69   ~ 0
+Text Notes 6500 4300 0    69   ~ 0
 Slew Rate is\nControlable
 Text Notes 6850 3600 0    69   ~ 0
@@
 3V3_C
 $Comp
-L GND #PWR070
+L GND #PWR77
 U 1 1 5604ED5E
 P 10000 4000
-F 0 "#PWR070" H 10000 3750 50  0001 C CNN
+F 0 "#PWR77" H 10000 3750 50  0001 C CNN
 F 1 "GND" H 10000 3850 50  0000 C CNN
 F 2 "" H 10000 4000 60  0000 C CNN
@@
 HUB_DP
 $Comp
-L GND #PWR071
+L GND #PWR76
 U 1 1 5604F800
 P 9850 2900
-F 0 "#PWR071" H 9850 2650 50  0001 C CNN
+F 0 "#PWR76" H 9850 2650 50  0001 C CNN
 F 1 "GND" V 9850 2700 50  0000 C CNN
 F 2 "" H 9850 2900 60  0000 C CNN
@@
 $EndComp
 $Comp
-L GND #PWR072
+L GND #PWR75
 U 1 1 5604F806
 P 9450 2700
-F 0 "#PWR072" H 9450 2450 50  0001 C CNN
+F 0 "#PWR75" H 9450 2450 50  0001 C CNN
 F 1 "GND" V 9450 2500 50  0000 C CNN
 F 2 "" H 9450 2700 60  0000 C CNN
@@
 Text Notes 8900 2150 0    60   ~ 0
 HUB Data, HOST Power
-Wire Notes Line
-	500  1850 10500 1850
 Wire Notes Line
 	10500 3350 500  3350
@@
 3V3_D
 $Comp
-L GND #PWR073
+L GND #PWR78
 U 1 1 56057D75
 P 10000 5000
-F 0 "#PWR073" H 10000 4750 50  0001 C CNN
+F 0 "#PWR78" H 10000 4750 50  0001 C CNN
 F 1 "GND" H 10000 4850 50  0000 C CNN
 F 2 "" H 10000 5000 60  0000 C CNN
@@
 Text GLabel 9200 4800 0    60   Input ~ 0
 3V3_A
-Text Notes 8700 5250 0    69   ~ 0
+Text Notes 8700 5300 0    69   ~ 0
 Slew Rate is\nControlable
 Text Notes 9250 3600 0    69   ~ 0
@@
 Text Notes 5200 2250 0    69   ~ 0
 HOST 5V0 rail
-Text Notes 8700 4250 0    69   ~ 0
+Text Notes 8700 4300 0    69   ~ 0
 Slew Rate is\nControlable
 $Comp
@@
 $EndComp
 $Comp
-L GND #PWR074
+L GND #PWR74
 U 1 1 561FF7A1
 P 8100 3100
-F 0 "#PWR074" H 8100 2850 50  0001 C CNN
+F 0 "#PWR74" H 8100 2850 50  0001 C CNN
 F 1 "GND" H 8100 2950 50  0000 C CNN
 F 2 "" H 8100 3100 60  0000 C CNN
@@
 HUB_PWR_PRT2
 $Comp
-L R R?
+L R R11
 U 1 1 5626E519
 P 5100 7400
-F 0 "R?" V 5180 7400 50  0000 C CNN
+F 0 "R11" V 5180 7400 50  0000 C CNN
 F 1 "0" V 5100 7400 50  0000 C CNN
 F 2 "Custom Parts:R_0603_sm" V 5030 7400 30  0001 C CNN
@@
 $EndComp
 $Comp
-L R R?
+L R R10
 U 1 1 5626E521
 P 5100 7250
-F 0 "R?" V 5180 7250 50  0000 C CNN
+F 0 "R10" V 5180 7250 50  0000 C CNN
 F 1 "DNS" V 5100 7250 50  0000 C CNN
 F 2 "Custom Parts:R_0603_sm" V 5030 7250 30  0001 C CNN
@@
 4V1_A
 $Comp
-L GND #PWR?
+L GND #PWR60
 U 1 1 5626E534
 P 2550 7650
-F 0 "#PWR?" H 2550 7400 50  0001 C CNN
+F 0 "#PWR60" H 2550 7400 50  0001 C CNN
 F 1 "GND" H 2550 7500 50  0000 C CNN
 F 2 "" H 2550 7650 60  0000 C CNN
@@
 12V0_B
 $Comp
-L CONN_02X10 P?
+L CONN_02X10 P18
 U 1 1 5626E544
 P 2800 7300
-F 0 "P?" H 2800 7750 50  0000 C CNN
+F 0 "P18" H 2800 7750 50  0000 C CNN
 F 1 "CONN_02X08" V 2800 7300 50  0000 C CNN
 F 2 "Pin_Headers:Pin_Header_Straight_2x10" H 2800 6100 60  0001 C CNN
@@
 12V0_B
 $Comp
-L GND #PWR?
+L GND #PWR64
 U 1 1 5626E54C
 P 3050 7650
-F 0 "#PWR?" H 3050 7400 50  0001 C CNN
+F 0 "#PWR64" H 3050 7400 50  0001 C CNN
 F 1 "GND" H 3050 7500 50  0000 C CNN
 F 2 "" H 3050 7650 60  0000 C CNN
@@
 $EndComp
 $Comp
-L GND #PWR?
+L GND #PWR63
 U 1 1 5626E552
 P 3050 6850
-F 0 "#PWR?" H 3050 6600 50  0001 C CNN
+F 0 "#PWR63" H 3050 6600 50  0001 C CNN
 F 1 "GND" H 3050 6700 50  0000 C CNN
 F 2 "" H 3050 6850 60  0000 C CNN
@@
 $EndComp
 $Comp
-L GND #PWR?
+L GND #PWR59
 U 1 1 5626E558
 P 2550 6850
-F 0 "#PWR?" H 2550 6600 50  0001 C CNN
+F 0 "#PWR59" H 2550 6600 50  0001 C CNN
 F 1 "GND" H 2550 6700 50  0000 C CNN
 F 2 "" H 2550 6850 60  0000 C CNN
@@
 Wire Notes Line
 	6250 6300 6250 6750
+Text GLabel 4900 750  0    60   Input ~ 0
+5V0_B_OUT
+Wire Wire Line
+	4900 750  4900 850
+Wire Wire Line
+	4900 1150 4900 1250
+$Comp
+L GND #PWR?
+U 1 1 5627A586
+P 4900 1550
+F 0 "#PWR?" H 4900 1300 50  0001 C CNN
+F 1 "GND" H 4900 1400 50  0000 C CNN
+F 2 "" H 4900 1550 60  0000 C CNN
+F 3 "" H 4900 1550 60  0000 C CNN
+	1    4900 1550
+	1    0    0    -1
+$EndComp
+Text GLabel 4900 1200 0    60   Input ~ 0
+HOST_SC
+Text Notes 5150 1600 0    60   ~ 0
+Short Circuit Detection\n5V0_B_OUT is post poly fuse\nSample using logic level (maybe A2D)\nLogic '0' signal (<1.5V) indicates poly\nfuse is set, host output is in protect.\nLogic '1' signal (approx 2.4V) indicates\npoly fuse is clear, normal opperation.\nAn A2D value that is too high might \nindicate the Host is not attached.
+$Comp
+L R R89
+U 1 1 5627A58F
+P 4900 1400
+F 0 "R89" V 4980 1400 50  0000 C CNN
+F 1 "47K" V 4900 1400 50  0000 C CNN
+F 2 "Custom Parts:R_0603_sm" V 4830 1400 30  0001 C CNN
+F 3 "http://www.mouser.com/ds/2/427/dcrcwe3-109170.pdf" H 4900 1400 30  0001 C CNN
+F 4 "71-CRCW0603-47K-E3" H 4900 1400 60  0001 C CNN "Mouse PN"
+	1    4900 1400
+	-1   0    0    1
+$EndComp
+$Comp
+L R R88
+U 1 1 5627A597
+P 4900 1000
+F 0 "R88" V 4980 1000 50  0000 C CNN
+F 1 "47K" V 4900 1000 50  0000 C CNN
+F 2 "Custom Parts:R_0603_sm" V 4830 1000 30  0001 C CNN
+F 3 "http://www.mouser.com/ds/2/427/dcrcwe3-109170.pdf" H 4900 1000 30  0001 C CNN
+F 4 "71-CRCW0603-47K-E3" H 4900 1000 60  0001 C CNN "Mouse PN"
+	1    4900 1000
+	-1   0    0    1
+$EndComp
+Wire Notes Line
+	3700 1850 3700 500
+Wire Notes Line
+	7750 1850 7750 500
+Wire Notes Line
+	7750 1850 10500 1850
+Wire Notes Line
+	3700 1850 500  1850
 $EndSCHEMATC
