File: Hardware/Make Files/Active/V2X.sch (KiCad schematic (older format))
At the start: 0 parts

Commit message: V2X V1.2 PCB build, with shares
Other:
- note removed: "All modules have switched power"
Changed lines of the file:
@@
 Text Notes 3150 3050 0    60   ~ 0
 enable
-Text Notes 1950 1000 0    60   ~ 0
-All modules have switched power
 Wire Notes Line
 	7500 4800 6750 4800
