File: Hardware/Make Files/Active/V2X_FTDI.sch (KiCad schematic (older format))
At the start: 25 parts, among them U1 FT4232H, U2 93C46, X1 12MHz

Commit message: home to work push
Parts:
- renumbered R3 to R2, R2 to R3
Other:
- note added: "FTDI ~RESET~ signal is \nautomatically controlled \nby HUB port enabled signal"
- moved on the sheet: R2, R3
Changed lines of the file:
@@
 F 0 "U1" H 5450 5400 50  0000 L CNN
 F 1 "FT4232H" H 7250 5400 50  0000 L CNN
-F 2 "Housings_QFP:LQFP-64_10x10mm_Pitch0.5mm" H 6500 3300 50  0000 C CNN
-F 3 "http://www.mouser.com/ds/2/163/DS_FT4232H-9150.pdf" H 6500 3300 50  0000 C CNN
+F 2 "Housings_QFP:LQFP-64_10x10mm_Pitch0.5mm" H 6500 3300 50  0001 C CNN
+F 3 "http://www.mouser.com/ds/2/163/DS_FT4232H-9150.pdf" H 6500 3300 50  0001 C CNN
 F 4 "895-FT4232HL" H 6500 3300 60  0001 C CNN "Mouse PN"
 	1    6500 3300
@@
 TXD\nRXD\n~RTS\n~CTS\n~DTR\n~DSR\n~DCD\n~RI
 $Comp
-L GND #PWR01
+L GND #PWR18
 U 1 1 55AD7D06
 P 7700 5000
-F 0 "#PWR01" H 7700 4750 50  0001 C CNN
+F 0 "#PWR18" H 7700 4750 50  0001 C CNN
 F 1 "GND" V 7700 4800 50  0000 C CNN
 F 2 "" H 7700 5000 60  0000 C CNN
@@
 $EndComp
 $Comp
-L GND #PWR02
+L GND #PWR17
 U 1 1 55AD7D39
 P 5900 5500
-F 0 "#PWR02" H 5900 5250 50  0001 C CNN
+F 0 "#PWR17" H 5900 5250 50  0001 C CNN
 F 1 "GND" V 5900 5300 50  0000 C CNN
 F 2 "" H 5900 5500 60  0000 C CNN
@@
 $EndComp
 $Comp
-L GND #PWR03
+L GND #PWR2
 U 1 1 55AD8749
 P 1200 3650
-F 0 "#PWR03" H 1200 3400 50  0001 C CNN
+F 0 "#PWR2" H 1200 3400 50  0001 C CNN
 F 1 "GND" H 1200 3500 50  0000 C CNN
 F 2 "" H 1200 3650 60  0000 C CNN
@@
 $EndComp
 $Comp
-L GND #PWR04
+L GND #PWR7
 U 1 1 55AD885E
 P 1700 1250
-F 0 "#PWR04" H 1700 1000 50  0001 C CNN
+F 0 "#PWR7" H 1700 1000 50  0001 C CNN
 F 1 "GND" H 1700 1100 50  0000 C CNN
 F 2 "" H 1700 1250 60  0000 C CNN
@@
 $EndComp
 $Comp
-L GND #PWR05
+L GND #PWR8
 U 1 1 55AD8999
 P 1700 2100
-F 0 "#PWR05" H 1700 1850 50  0001 C CNN
+F 0 "#PWR8" H 1700 1850 50  0001 C CNN
 F 1 "GND" H 1700 1950 50  0000 C CNN
 F 2 "" H 1700 2100 60  0000 C CNN
@@
 $EndComp
 $Comp
-L GND #PWR06
+L GND #PWR1
 U 1 1 55AD8CCE
 P 1050 2850
-F 0 "#PWR06" H 1050 2600 50  0001 C CNN
+F 0 "#PWR1" H 1050 2600 50  0001 C CNN
 F 1 "GND" H 1050 2700 50  0000 C CNN
 F 2 "" H 1050 2850 60  0000 C CNN
@@
 Power Filtering
 $Comp
-L GND #PWR07
+L GND #PWR15
 U 1 1 55AD97DA
 P 4800 2700
-F 0 "#PWR07" H 4800 2450 50  0001 C CNN
+F 0 "#PWR15" H 4800 2450 50  0001 C CNN
 F 1 "GND" V 4800 2500 50  0000 C CNN
 F 2 "" H 4800 2700 60  0000 C CNN
@@
 EECLK
 $Comp
-L GND #PWR08
+L GND #PWR5
 U 1 1 55ADAE78
 P 1550 7500
-F 0 "#PWR08" H 1550 7250 50  0001 C CNN
+F 0 "#PWR5" H 1550 7250 50  0001 C CNN
 F 1 "GND" V 1550 7300 50  0000 C CNN
 F 2 "" H 1550 7500 60  0000 C CNN
@@
 FTDI Device Configuration EEPROM
 $Comp
-L GND #PWR09
+L GND #PWR10
 U 1 1 55ADBFB3
 P 1950 1250
-F 0 "#PWR09" H 1950 1000 50  0001 C CNN
+F 0 "#PWR10" H 1950 1000 50  0001 C CNN
 F 1 "GND" H 1950 1100 50  0000 C CNN
 F 2 "" H 1950 1250 60  0000 C CNN
@@
 $EndComp
 $Comp
-L GND #PWR010
+L GND #PWR11
 U 1 1 55ADBFF1
 P 1950 2100
-F 0 "#PWR010" H 1950 1850 50  0001 C CNN
+F 0 "#PWR11" H 1950 1850 50  0001 C CNN
 F 1 "GND" H 1950 1950 50  0000 C CNN
 F 2 "" H 1950 2100 60  0000 C CNN
@@
 $EndComp
 $Comp
-L GND #PWR011
+L GND #PWR4
 U 1 1 55ADC2B9
 P 1500 3650
-F 0 "#PWR011" H 1500 3400 50  0001 C CNN
+F 0 "#PWR4" H 1500 3400 50  0001 C CNN
 F 1 "GND" H 1500 3500 50  0000 C CNN
 F 2 "" H 1500 3650 60  0000 C CNN
@@
 $EndComp
 $Comp
-L GND #PWR012
+L GND #PWR3
 U 1 1 55ADC2C5
 P 1350 2850
-F 0 "#PWR012" H 1350 2600 50  0001 C CNN
+F 0 "#PWR3" H 1350 2600 50  0001 C CNN
 F 1 "GND" H 1350 2700 50  0000 C CNN
 F 2 "" H 1350 2850 60  0000 C CNN
@@
 $EndComp
 $Comp
-L GND #PWR013
+L GND #PWR9
 U 1 1 55ADC34F
 P 1800 3650
-F 0 "#PWR013" H 1800 3400 50  0001 C CNN
+F 0 "#PWR9" H 1800 3400 50  0001 C CNN
 F 1 "GND" H 1800 3500 50  0000 C CNN
 F 2 "" H 1800 3650 60  0000 C CNN
@@
 $EndComp
 $Comp
-L GND #PWR014
+L GND #PWR6
 U 1 1 55ADC35B
 P 1650 2850
-F 0 "#PWR014" H 1650 2600 50  0001 C CNN
+F 0 "#PWR6" H 1650 2600 50  0001 C CNN
 F 1 "GND" H 1650 2700 50  0000 C CNN
 F 2 "" H 1650 2850 60  0000 C CNN
@@
 $EndComp
 $Comp
-L GND #PWR015
+L GND #PWR12
 U 1 1 55ADC37F
 P 1950 2850
-F 0 "#PWR015" H 1950 2600 50  0001 C CNN
+F 0 "#PWR12" H 1950 2600 50  0001 C CNN
 F 1 "GND" H 1950 2700 50  0000 C CNN
 F 2 "" H 1950 2850 60  0000 C CNN
@@
 $EndComp
 $Comp
-L GND #PWR016
+L GND #PWR13
 U 1 1 55ADC373
 P 2100 3650
-F 0 "#PWR016" H 2100 3400 50  0001 C CNN
+F 0 "#PWR13" H 2100 3400 50  0001 C CNN
 F 1 "GND" H 2100 3500 50  0000 C CNN
 F 2 "" H 2100 3650 60  0000 C CNN
@@
 $EndComp
 $Comp
-L GND #PWR017
+L GND #PWR14
 U 1 1 55ADC68C
 P 2250 2850
-F 0 "#PWR017" H 2250 2600 50  0001 C CNN
+F 0 "#PWR14" H 2250 2600 50  0001 C CNN
 F 1 "GND" H 2250 2700 50  0000 C CNN
 F 2 "" H 2250 2850 60  0000 C CNN
@@
 Text GLabel 5300 2500 0    67   Input ~ 0
 FTDI_DP
-Text GLabel 4350 2900 0    60   Input ~ 0
+Text GLabel 4800 2900 0    60   Input ~ 0
 ~FTDI_RESET
 Text GLabel 900  950  0    60   Input ~ 0
@@
 Text Notes 9150 3250 0    60   ~ 0
 Serial channel for Accelerometer data\n
-Text GLabel 4350 3050 0    69   Input ~ 0
+Text GLabel 4800 3050 0    69   Input ~ 0
 HUB_PWR_PRT1
 $Comp
-L R R3
+L R R2
 U 1 1 5606A910
-P 4500 3050
-F 0 "R3" V 4580 3050 50  0000 C CNN
-F 1 "DNS" V 4500 3050 50  0000 C CNN
-F 2 "Custom Parts:R_0603_sm" V 4430 3050 30  0001 C CNN
-F 3 "" H 4500 3050 30  0000 C CNN
-	1    4500 3050
+P 4950 2900
+F 0 "R2" V 5030 2900 50  0000 C CNN
+F 1 "DNS" V 4950 2900 50  0000 C CNN
+F 2 "Custom Parts:R_0603_sm" V 4880 2900 30  0001 C CNN
+F 3 "" H 4950 2900 30  0000 C CNN
+	1    4950 2900
 	0    1    1    0
 $EndComp
@@
 	7700 1500 8050 1500
 Wire Wire Line
-	4650 3050 4700 3050
-Wire Wire Line
-	4700 3050 4700 2900
-Wire Wire Line
-	4650 2900 5300 2900
-Connection ~ 4700 2900
+	5100 3050 5150 3050
+Wire Wire Line
+	5150 3050 5150 2900
+Wire Wire Line
+	5100 2900 5300 2900
+Connection ~ 5150 2900
 $Comp
 L FILTER FB2
@@
 3V3_B
 $Comp
-L R R2
+L R R3
 U 1 1 56090D92
-P 4500 2900
-F 0 "R2" V 4580 2900 50  0000 C CNN
-F 1 "0" V 4500 2900 50  0000 C CNN
-F 2 "Custom Parts:R_0603_sm" V 4430 2900 30  0001 C CNN
-F 3 "http://www.mouser.com/ds/2/427/dcrcwe3-109170.pdf" H 4500 2900 30  0001 C CNN
-F 4 "71-CRCW0603-0-E3" H 4500 2900 60  0001 C CNN "Mouse PN"
-	1    4500 2900
+P 4950 3050
+F 0 "R3" V 5030 3050 50  0000 C CNN
+F 1 "0" V 4950 3050 50  0000 C CNN
+F 2 "Custom Parts:R_0603_sm" V 4880 3050 30  0001 C CNN
+F 3 "http://www.mouser.com/ds/2/427/dcrcwe3-109170.pdf" H 4950 3050 30  0001 C CNN
+F 4 "71-CRCW0603-0-E3" H 4950 3050 60  0001 C CNN "Mouse PN"
+	1    4950 3050
 	0    -1   1    0
 $EndComp
 $Comp
-L GND #PWR018
+L GND #PWR16
 U 1 1 55B7E844
 P 5350 6950
-F 0 "#PWR018" H 5350 6700 50  0001 C CNN
+F 0 "#PWR16" H 5350 6700 50  0001 C CNN
 F 1 "GND" H 5350 6800 50  0000 C CNN
 F 2 "" H 5350 6950 60  0000 C CNN
@@
 Wire Wire Line
 	6000 1050 6000 1100
+Text Notes 3750 3500 0    69   ~ 0
+FTDI ~RESET~ signal is \nautomatically controlled \nby HUB port enabled signal
 $EndSCHEMATC

Commit message: V2X V1.2 PCB build, with shares
Parts:
- U1: symbol FT4232H -> FT4232H-RESCUE-V2X
Connections:
- no-connect marks 0 -> 26
Changed lines of the file:
@@
 $EndDescr
 $Comp
-L FT4232H U1
+L FT4232H-RESCUE-V2X U1
 U 1 1 55AD78AF
 P 6500 3300
@@
 Text Notes 3750 3500 0    69   ~ 0
 FTDI ~RESET~ signal is \nautomatically controlled \nby HUB port enabled signal
+NoConn ~ 7700 1600
+NoConn ~ 7700 1700
+NoConn ~ 7700 1800
+NoConn ~ 7700 1900
+NoConn ~ 7700 2000
+NoConn ~ 7700 2100
+NoConn ~ 7700 2500
+NoConn ~ 7700 2600
+NoConn ~ 7700 2700
+NoConn ~ 7700 2800
+NoConn ~ 7700 2900
+NoConn ~ 7700 3000
+NoConn ~ 7700 3400
+NoConn ~ 7700 3500
+NoConn ~ 7700 3600
+NoConn ~ 7700 3700
+NoConn ~ 7700 3800
+NoConn ~ 7700 3900
+NoConn ~ 7700 4100
+NoConn ~ 7700 4200
+NoConn ~ 7700 4300
+NoConn ~ 7700 4400
+NoConn ~ 7700 4500
+NoConn ~ 7700 4600
+NoConn ~ 7700 4700
+NoConn ~ 7700 4800
 $EndSCHEMATC

Commit message: BOM updates
Parts:
- C1, C3: Mouse PN 963-LMK212B7475KG-T -> 581-12063C475KAT2A
Changed lines of the file:
@@
 F 2 "Custom Parts:C_0805_SM" H 1738 950 30  0001 C CNN
 F 3 "http://www.yuden.co.jp/productdata/catalog/en/mlcc_all_e.pdf" H 1700 1100 60  0001 C CNN
-F 4 "963-LMK212B7475KG-T" H 1700 1100 60  0001 C CNN "Mouse PN"
+F 4 "581-12063C475KAT2A" H 1700 1100 60  0001 C CNN "Mouse PN"
 	1    1700 1100
 	-1   0    0    -1
@@
 F 2 "Custom Parts:C_0805_SM" H 1738 1800 30  0001 C CNN
 F 3 "http://www.yuden.co.jp/productdata/catalog/en/mlcc_all_e.pdf" H 1700 1950 60  0001 C CNN
-F 4 "963-LMK212B7475KG-T" H 1700 1950 60  0001 C CNN "Mouse PN"
+F 4 "581-12063C475KAT2A" H 1700 1950 60  0001 C CNN "Mouse PN"
 	1    1700 1950
 	-1   0    0    -1
