File: Hardware/Make Files/Active/_autosave-V2X.kicad_pcb (KiCad board)
At the start: 2 copper layers, 85 x 56 mm, 224 parts, among them CON1 AVR-PDI-6, J1 DB9, P10 Board Mount 2, P11 Ficudial2, P12 Board Mount 3, P13 Ficudial3, P15 Board Mount 4, P16 Ficudial4, P17 CUR_SEN, P18 CONN_02X08, P19 CUR_SEN, P20 Jumper 1, P21 Jumper 2, P22 CONN_02X04, P23 Jumper 3, P24 Jumper 4, P5 NVM_RST, P6 Board Mount 1, P7 Ficudial1, P8 USB_A, P9 USB_u, Q1 2N7000, Q10 2N3904, Q11 IRF9335, Q13 BSS84, Q14 IRF9335, Q15 2N7000, Q16 2N7000, Q17 2N7000, Q18 2N7000, Q19 2N7000, Q2 BSS84, Q3 BSS84, Q4 BSS84, Q5 3906, Q6 2N3904, Q7 2N7000, Q8 2N3904, Q9 2N3904, SW1 SPST, SW2 SW_PUSH, U1 FT4232H, U10 MCP2551, U11 XRP6124, U12 SLG59M, U14 ATXMEGA16A4U-A, U15 SLG59M, U16 SLG59M, U17 XRP6124, U18 SLG59M, U19 ADXL345, U2 93C46, U20 USB2242, U21 74LS126, U22 74HC595, U23 74HC595, U5 ESDAxxSC6, U6 ESDAxxSC6, U7 STN1110, U8 LM339, U9 LM317, X1 12MHz, X2 16MHz, X3 24MHz

Commit message: Project Shares and Next rev cleanup
Routing:
- net GND: track 693.5 -> 696.1 mm
Changed lines of the file:
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@@
     (thickness 1.6)
     (drawings 24)
-    (tracks 3409)
+    (tracks 3411)
     (zones 0)
     (modules 224)
@@
       (drillshape 0)
       (scaleselection 1)
-      (outputdirectory C:/Users/jbanks2/Documents/Projects/rvi_v2x_board/Hardware/Gerbers/Active/))
+      (outputdirectory "C:/Users/jbanks2/Documents/Projects/rvi_v2x_board/Hardware/Project Shares/V1.2/"))
   )
   (net 0 "")
@@
   (segment (start 86.95 137.25) (end 85.55 137.25) (width 0.25) (layer F.Cu) (net 1))
   (segment (start 84.25 137.5) (end 82.95 137.5) (width 0.25) (layer B.Cu) (net 1))
+  (segment (start 52.65 155.3) (end 51.6 154.25) (width 0.25) (layer F.Cu) (net 2))
+  (segment (start 52.65 156.7) (end 52.65 155.3) (width 0.25) (layer F.Cu) (net 2))
+  (segment (start 52.15 152.55) (end 52.25 152.45) (width 0.25) (layer B.Cu) (net 2))
+  (segment (start 52.15 152.6) (end 52.15 152.55) (width 0.25) (layer B.Cu) (net 2))
+  (via (at 52.15 152.6) (size 0.6) (drill 0.4) (layers F.Cu B.Cu) (net 2))
+  (segment (start 51.6 153.15) (end 52.15 152.6) (width 0.25) (layer F.Cu) (net 2))
+  (segment (start 51.6 154.25) (end 51.6 153.15) (width 0.25) (layer F.Cu) (net 2))
   (segment (start 79 170.535) (end 79 168.6) (width 0.25) (layer F.Cu) (net 2))
   (segment (start 79 168.6) (end 79 168.5) (width 0.25) (layer F.Cu) (net 2))
@@
   (segment (start 62.55 143.9) (end 62.75 143.9) (width 0.25) (layer B.Cu) (net 2))
   (via (at 62.55 143.9) (size 0.6) (drill 0.4) (layers F.Cu B.Cu) (net 2))
-  (segment (start 52.65 156.7) (end 52.65 155.3) (width 0.25) (layer F.Cu) (net 2))
-  (segment (start 52.25 152.5) (end 52.35 152.5) (width 0.25) (layer B.Cu) (net 2))
-  (segment (start 52.15 152.6) (end 52.25 152.5) (width 0.25) (layer B.Cu) (net 2))
-  (via (at 52.15 152.6) (size 0.6) (drill 0.4) (layers F.Cu B.Cu) (net 2))
-  (segment (start 51.65 153.1) (end 52.15 152.6) (width 0.25) (layer F.Cu) (net 2))
   (segment (start 51.75 170.1) (end 52.95 170.1) (width 0.25) (layer F.Cu) (net 2))
   (segment (start 52.95 170.1) (end 52.95 170.3) (width 0.25) (layer B.Cu) (net 2))
@@
   (segment (start 50.45 167.7) (end 50.95 168.2) (width 0.25) (layer B.Cu) (net 25))
   (segment (start 50.45 166.2) (end 50.45 167.7) (width 0.25) (layer B.Cu) (net 25))
-  (segment (start 50.25 154.5) (end 50.25 153.9) (width 0.25) (layer B.Cu) (net 25) (status 800000))
-  (segment (start 50.25 153.9) (end 50.2 153.9) (width 0.25) (layer B.Cu) (net 25) (status C00000))
-  (segment (start 50.2 153.9) (end 48.8 152.5) (width 0.25) (layer B.Cu) (net 25) (status 400000))
+  (segment (start 50.25 154.5) (end 50.25 153.9) (width 0.25) (layer B.Cu) (net 25))
+  (segment (start 50.25 153.9) (end 50.2 153.9) (width 0.25) (layer B.Cu) (net 25))
+  (segment (start 50.2 153.9) (end 48.8 152.5) (width 0.25) (layer B.Cu) (net 25))
   (segment (start 49.05 150.65) (end 49.05 147.6) (width 0.25) (layer F.Cu) (net 25))
   (segment (start 48.8 150.9) (end 49.05 150.65) (width 0.25) (layer F.Cu) (net 25))
@@
   (segment (start 40.25 143.9) (end 38.4 143.9) (width 0.5) (layer F.Cu) (net 158))
   (segment (start 38.4 143.9) (end 38.25 144.05) (width 0.5) (layer F.Cu) (net 158))
-  (segment (start 38.25 144.05) (end 38.25 143.05) (width 0.25) (layer B.Cu) (net 159) (status 400000))
-  (segment (start 38.25 142.95) (end 38.25 141.95) (width 0.25) (layer F.Cu) (net 159) (status 800000))
+  (segment (start 38.25 144.05) (end 38.25 143.05) (width 0.25) (layer B.Cu) (net 159))
+  (segment (start 38.25 142.95) (end 38.25 141.95) (width 0.25) (layer F.Cu) (net 159))
   (segment (start 38.3 143) (end 38.25 142.95) (width 0.25) (layer F.Cu) (net 159))
   (via (at 38.3 143) (size 0.6) (drill 0.4) (layers F.Cu B.Cu) (net 159))
   (segment (start 38.25 143.05) (end 38.3 143) (width 0.25) (layer B.Cu) (net 159))
-  (segment (start 40.25 143.9) (end 38.4 143.9) (width 0.25) (layer B.Cu) (net 159) (status C00000))
-  (segment (start 38.4 143.9) (end 38.25 144.05) (width 0.25) (layer B.Cu) (net 159) (status C00000))
+  (segment (start 40.25 143.9) (end 38.4 143.9) (width 0.25) (layer B.Cu) (net 159))
+  (segment (start 38.4 143.9) (end 38.25 144.05) (width 0.25) (layer B.Cu) (net 159))
   (segment (start 40.25 143.9) (end 40.45 143.9) (width 0.25) (layer B.Cu) (net 159))
-  (segment (start 42.25 142.1) (end 40.25 142.1) (width 0.25) (layer B.Cu) (net 160) (status C00000))
+  (segment (start 42.25 142.1) (end 40.25 142.1) (width 0.25) (layer B.Cu) (net 160))
   (segment (start 38.75 146.45098) (end 41.60098 146.45098) (width 0.25) (layer F.Cu) (net 161))
   (segment (start 41.60098 146.45098) (end 41.75 146.6) (width 0.25) (layer F.Cu) (net 161))
