File: Hardware/Make Files/Active/V2X_PWR.sch (KiCad schematic (older format))
At the start: 60 parts, among them P10 Board Mount 2, P11 Ficudial2, P12 Board Mount 3, P13 Ficudial3, P15 Board Mount 4, P16 Ficudial4, P17 CUR_SEN, P18 CONN_02X08, P19 CUR_SEN, P6 Board Mount 1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

Commit message: V2X V1.2 PCB build, with shares
Parts:
- added C65: 10N, Custom Parts:C_0603_SM, symbol C
- added P25: Ficudial1, Fiducials:Fiducial_1mm_Dia_2.54mm_Outer_CopperTop, symbol CONN_01X01
- added P27: Ficudial2, Fiducials:Fiducial_1mm_Dia_2.54mm_Outer_CopperTop, symbol CONN_01X01
- added P28: Ficudial3, Fiducials:Fiducial_1mm_Dia_2.54mm_Outer_CopperTop, symbol CONN_01X01
- added P29: Ficudial4, Fiducials:Fiducial_1mm_Dia_2.54mm_Outer_CopperTop, symbol CONN_01X01
- D11: value SD15C -> SMBJ16A; footprint Diodes_SMD:SOD-323 -> Diodes_SMD:SMB_Standard; Mouse PN 576-SD15C-01FTG -> 511-SMBJ16A
- SW2: symbol SW_PUSH -> SW_PUSH_SLD
Connections:
- wire segments 54 -> 55
- no-connect marks 0 -> 15
Other:
- moved on the sheet: P10, P11, P12, P13, P15, P16, P6, P7
Changed lines of the file:
@@
 P 2400 1300
 F 0 "D11" H 2400 1450 50  0000 C CNN
-F 1 "SD15C" H 2400 1150 50  0000 C CNN
-F 2 "Diodes_SMD:SOD-323" H 2400 1300 60  0001 C CNN
-F 3 "http://www.mouser.com/ds/2/240/littelfuse_SD-C_datasheet-341330.pdf" H 2400 1300 60  0001 C CNN
-F 4 "576-SD15C-01FTG" H 2400 1300 60  0001 C CNN "Mouse PN"
+F 1 "SMBJ16A" H 2400 1150 50  0000 C CNN
+F 2 "Diodes_SMD:SMB_Standard" H 2400 1300 60  0001 C CNN
+F 3 "http://www.mouser.com/ds/2/389/CD00001366-310691.pdf" H 2400 1300 60  0001 C CNN
+F 4 "511-SMBJ16A" H 2400 1300 60  0001 C CNN "Mouse PN"
 	1    2400 1300
 	0    1    1    0
@@
 L CONN_01X01 P7
 U 1 1 55C35919
-P 9550 800
-F 0 "P7" H 9550 900 50  0000 C CNN
-F 1 "Ficudial1" H 9550 700 50  0000 C CNN
-F 2 "Fiducials:Fiducial_1mm_Dia_2.54mm_Outer_CopperTop" H 9550 800 60  0001 C CNN
-F 3 "" H 9550 800 60  0000 C CNN
-	1    9550 800
+P 8900 800
+F 0 "P7" H 8900 900 50  0000 C CNN
+F 1 "Ficudial1" H 8900 700 50  0000 C CNN
+F 2 "Fiducials:Fiducial_1mm_Dia_2.54mm_Outer_CopperTop" H 8900 800 60  0001 C CNN
+F 3 "" H 8900 800 60  0000 C CNN
+	1    8900 800
 	-1   0    0    1
 $EndComp
@@
 L CONN_01X01 P11
 U 1 1 55C35920
-P 9550 1050
-F 0 "P11" H 9550 1150 50  0000 C CNN
-F 1 "Ficudial2" H 9550 950 50  0000 C CNN
-F 2 "Fiducials:Fiducial_1mm_Dia_2.54mm_Outer_CopperTop" H 9550 1050 60  0001 C CNN
-F 3 "" H 9550 1050 60  0000 C CNN
-	1    9550 1050
+P 8900 1050
+F 0 "P11" H 8900 1150 50  0000 C CNN
+F 1 "Ficudial2" H 8900 950 50  0000 C CNN
+F 2 "Fiducials:Fiducial_1mm_Dia_2.54mm_Outer_CopperTop" H 8900 1050 60  0001 C CNN
+F 3 "" H 8900 1050 60  0000 C CNN
+	1    8900 1050
 	-1   0    0    1
 $EndComp
@@
 L CONN_01X01 P13
 U 1 1 55C35927
-P 9550 1300
-F 0 "P13" H 9550 1400 50  0000 C CNN
-F 1 "Ficudial3" H 9550 1200 50  0000 C CNN
-F 2 "Fiducials:Fiducial_1mm_Dia_2.54mm_Outer_CopperTop" H 9550 1300 60  0001 C CNN
-F 3 "" H 9550 1300 60  0000 C CNN
-	1    9550 1300
+P 8900 1300
+F 0 "P13" H 8900 1400 50  0000 C CNN
+F 1 "Ficudial3" H 8900 1200 50  0000 C CNN
+F 2 "Fiducials:Fiducial_1mm_Dia_2.54mm_Outer_CopperTop" H 8900 1300 60  0001 C CNN
+F 3 "" H 8900 1300 60  0000 C CNN
+	1    8900 1300
 	-1   0    0    1
 $EndComp
@@
 L CONN_01X01 P16
 U 1 1 55C3592E
-P 9550 1550
-F 0 "P16" H 9550 1650 50  0000 C CNN
-F 1 "Ficudial4" H 9550 1450 50  0000 C CNN
-F 2 "Fiducials:Fiducial_1mm_Dia_2.54mm_Outer_CopperTop" H 9550 1550 60  0001 C CNN
-F 3 "" H 9550 1550 60  0000 C CNN
-	1    9550 1550
+P 8900 1550
+F 0 "P16" H 8900 1650 50  0000 C CNN
+F 1 "Ficudial4" H 8900 1450 50  0000 C CNN
+F 2 "Fiducials:Fiducial_1mm_Dia_2.54mm_Outer_CopperTop" H 8900 1550 60  0001 C CNN
+F 3 "" H 8900 1550 60  0000 C CNN
+	1    8900 1550
 	-1   0    0    1
 $EndComp
@@
 L CONN_01X01 P6
 U 1 1 55C35935
-P 9000 800
-F 0 "P6" H 9000 900 50  0000 C CNN
-F 1 "Board Mount 1" H 9000 700 50  0000 C CNN
-F 2 "Mounting_Holes:MountingHole_3mm" H 9000 800 60  0001 C CNN
-F 3 "" H 9000 800 60  0000 C CNN
-	1    9000 800
+P 8150 800
+F 0 "P6" H 8150 900 50  0000 C CNN
+F 1 "Board Mount 1" H 8150 700 50  0000 C CNN
+F 2 "Mounting_Holes:MountingHole_3mm" H 8150 800 60  0001 C CNN
+F 3 "" H 8150 800 60  0000 C CNN
+	1    8150 800
 	-1   0    0    1
 $EndComp
@@
 L CONN_01X01 P10
 U 1 1 55C3593C
-P 9000 1050
-F 0 "P10" H 9000 1150 50  0000 C CNN
-F 1 "Board Mount 2" H 9000 950 50  0000 C CNN
-F 2 "Mounting_Holes:MountingHole_3mm" H 9000 1050 60  0001 C CNN
-F 3 "" H 9000 1050 60  0000 C CNN
-	1    9000 1050
+P 8150 1050
+F 0 "P10" H 8150 1150 50  0000 C CNN
+F 1 "Board Mount 2" H 8150 950 50  0000 C CNN
+F 2 "Mounting_Holes:MountingHole_3mm" H 8150 1050 60  0001 C CNN
+F 3 "" H 8150 1050 60  0000 C CNN
+	1    8150 1050
 	-1   0    0    1
 $EndComp
@@
 L CONN_01X01 P12
 U 1 1 55C35943
-P 9000 1300
-F 0 "P12" H 9000 1400 50  0000 C CNN
-F 1 "Board Mount 3" H 9000 1200 50  0000 C CNN
-F 2 "Mounting_Holes:MountingHole_3mm" H 9000 1300 60  0001 C CNN
-F 3 "" H 9000 1300 60  0000 C CNN
-	1    9000 1300
+P 8150 1300
+F 0 "P12" H 8150 1400 50  0000 C CNN
+F 1 "Board Mount 3" H 8150 1200 50  0000 C CNN
+F 2 "Mounting_Holes:MountingHole_3mm" H 8150 1300 60  0001 C CNN
+F 3 "" H 8150 1300 60  0000 C CNN
+	1    8150 1300
 	-1   0    0    1
 $EndComp
@@
 L CONN_01X01 P15
 U 1 1 55C3594A
-P 9000 1550
-F 0 "P15" H 9000 1650 50  0000 C CNN
-F 1 "Board Mount 4" H 9000 1450 50  0000 C CNN
-F 2 "Mounting_Holes:MountingHole_3mm" H 9000 1550 60  0001 C CNN
-F 3 "" H 9000 1550 60  0000 C CNN
-	1    9000 1550
+P 8150 1550
+F 0 "P15" H 8150 1650 50  0000 C CNN
+F 1 "Board Mount 4" H 8150 1450 50  0000 C CNN
+F 2 "Mounting_Holes:MountingHole_3mm" H 8150 1550 60  0001 C CNN
+F 3 "" H 8150 1550 60  0000 C CNN
+	1    8150 1550
 	-1   0    0    1
 $EndComp
@@
 3V3_EN
 $Comp
-L SW_PUSH SW2
+L SW_PUSH_SLD SW2
 U 1 1 5600CE81
 P 2200 4900
@@
 	1    0    0    -1
 $EndComp
-Text GLabel 2150 4550 2    69   Input ~ 0
+Text GLabel 2550 4550 2    69   Input ~ 0
 BUTTON
 Wire Wire Line
@@
 Wire Wire Line
 	3400 4450 3500 4450
-Text Notes 800  5500 0    69   ~ 0
+Text Notes 800  5600 0    69   ~ 0
 Button force starts the 3V3 to start SEQ\nSEQ must hold 3V3_EN high to stay on\nBUTTON is soft button signal once running\n3V3_EN pulled low kills supply regaurdless if button pressed
 Wire Wire Line
@@
 Text GLabel 3050 6850 2    69   Input ~ 0
 SIM_WAKE
+$Comp
+L C C65
+U 1 1 56290CF9
+P 2300 4400
+F 0 "C65" H 2325 4500 50  0000 L CNN
+F 1 "10N" H 2325 4300 50  0000 L CNN
+F 2 "Custom Parts:C_0603_SM" H 2338 4250 30  0001 C CNN
+F 3 "http://www.mouser.com/ds/2/427/vjw1bcbascomseries-223529.pdf" H 2300 4400 60  0001 C CNN
+F 4 "77-VJ0603Y103KXACBC" H 2300 4400 60  0001 C CNN "Mouse PN"
+	1    2300 4400
+	1    0    0    -1
+$EndComp
+Wire Wire Line
+	2150 4550 2550 4550
+Connection ~ 2300 4550
+$Comp
+L GND #PWR079
+U 1 1 562917CA
+P 2300 4250
+F 0 "#PWR079" H 2300 4000 50  0001 C CNN
+F 1 "GND" V 2400 4200 50  0000 C CNN
+F 2 "" H 2300 4250 60  0000 C CNN
+F 3 "" H 2300 4250 60  0000 C CNN
+	1    2300 4250
+	-1   0    0    1
+$EndComp
+$Comp
+L GND #PWR080
+U 1 1 562939B7
+P 1900 5000
+F 0 "#PWR080" H 1900 4750 50  0001 C CNN
+F 1 "GND" H 1900 4850 50  0000 C CNN
+F 2 "" H 1900 5000 60  0000 C CNN
+F 3 "" H 1900 5000 60  0000 C CNN
+	1    1900 5000
+	1    0    0    -1
+$EndComp
+$Comp
+L CONN_01X01 P25
+U 1 1 562955D0
+P 9400 800
+F 0 "P25" H 9400 900 50  0000 C CNN
+F 1 "Ficudial1" H 9400 700 50  0000 C CNN
+F 2 "Fiducials:Fiducial_1mm_Dia_2.54mm_Outer_CopperTop" H 9400 800 60  0001 C CNN
+F 3 "" H 9400 800 60  0000 C CNN
+	1    9400 800
+	-1   0    0    1
+$EndComp
+$Comp
+L CONN_01X01 P27
+U 1 1 562955D6
+P 9400 1050
+F 0 "P27" H 9400 1150 50  0000 C CNN
+F 1 "Ficudial2" H 9400 950 50  0000 C CNN
+F 2 "Fiducials:Fiducial_1mm_Dia_2.54mm_Outer_CopperTop" H 9400 1050 60  0001 C CNN
+F 3 "" H 9400 1050 60  0000 C CNN
+	1    9400 1050
+	-1   0    0    1
+$EndComp
+$Comp
+L CONN_01X01 P28
+U 1 1 562955DC
+P 9400 1300
+F 0 "P28" H 9400 1400 50  0000 C CNN
+F 1 "Ficudial3" H 9400 1200 50  0000 C CNN
+F 2 "Fiducials:Fiducial_1mm_Dia_2.54mm_Outer_CopperTop" H 9400 1300 60  0001 C CNN
+F 3 "" H 9400 1300 60  0000 C CNN
+	1    9400 1300
+	-1   0    0    1
+$EndComp
+$Comp
+L CONN_01X01 P29
+U 1 1 562955E2
+P 9400 1550
+F 0 "P29" H 9400 1650 50  0000 C CNN
+F 1 "Ficudial4" H 9400 1450 50  0000 C CNN
+F 2 "Fiducials:Fiducial_1mm_Dia_2.54mm_Outer_CopperTop" H 9400 1550 60  0001 C CNN
+F 3 "" H 9400 1550 60  0000 C CNN
+	1    9400 1550
+	-1   0    0    1
+$EndComp
+NoConn ~ 9100 800
+NoConn ~ 9100 1050
+NoConn ~ 9100 1300
+NoConn ~ 9100 1550
+NoConn ~ 9600 1550
+NoConn ~ 9600 1300
+NoConn ~ 9600 1050
+NoConn ~ 9600 800
+NoConn ~ 7700 2700
+NoConn ~ 7700 2800
+NoConn ~ 9450 2600
+NoConn ~ 8350 800
+NoConn ~ 8350 1050
+NoConn ~ 8350 1300
+NoConn ~ 8350 1550
 $EndSCHEMATC

Commit message: BOM updates
Parts:
- P18: value CONN_02X08 -> CONN_02X10
- P8: Mouse PN (none) -> 523-UE27AC5410H
- R10: Mouse PN 71-CRCW0603-22.1-E3 -> (none)
- R70, R73: value 10K5 -> 10K; Mouse PN 71-CRCW0603-10.5k-E3 -> 71-CRCW0603-10k-E3
Changed lines of the file:
@@
 P 2000 4150
 F 0 "R70" V 2080 4150 50  0000 C CNN
-F 1 "10K5" V 2000 4150 50  0000 C CNN
+F 1 "10K" V 2000 4150 50  0000 C CNN
 F 2 "Custom Parts:R_0603_sm" V 1930 4150 30  0001 C CNN
 F 3 "http://www.mouser.com/ds/2/427/dcrcwe3-109170.pdf" H 2000 4150 30  0001 C CNN
-F 4 "71-CRCW0603-10.5k-E3" H 2000 4150 60  0001 C CNN "Mouse PN"
+F 4 "71-CRCW0603-10k-E3" H 2000 4150 60  0001 C CNN "Mouse PN"
 	1    2000 4150
 	1    0    0    1
@@
 P 1700 4750
 F 0 "R73" V 1780 4750 50  0000 C CNN
-F 1 "10K5" V 1700 4750 50  0000 C CNN
+F 1 "10K" V 1700 4750 50  0000 C CNN
 F 2 "Custom Parts:R_0603_sm" V 1630 4750 30  0001 C CNN
 F 3 "http://www.mouser.com/ds/2/427/dcrcwe3-109170.pdf" H 1700 4750 30  0001 C CNN
-F 4 "71-CRCW0603-10.5k-E3" H 1700 4750 60  0001 C CNN "Mouse PN"
+F 4 "71-CRCW0603-10k-E3" H 1700 4750 60  0001 C CNN "Mouse PN"
 	1    1700 4750
 	1    0    0    1
@@
 F 1 "USB_A" H 7950 3000 50  0000 C CNN
 F 2 "Connect:USB_A" V 7950 2700 60  0001 C CNN
-F 3 "" V 7950 2700 60  0000 C CNN
+F 3 "http://www.mouser.com/ds/2/18/USB_CAT-274878.pdf" V 7950 2700 60  0001 C CNN
+F 4 "523-UE27AC5410H" H 8000 2800 60  0001 C CNN "Mouse PN"
 	1    8000 2800
 	0    1    1    0
@@
 F 1 "DNS" V 5100 7250 50  0000 C CNN
 F 2 "Custom Parts:R_0603_sm" V 5030 7250 30  0001 C CNN
-F 3 "http://www.mouser.com/ds/2/427/dcrcwe3-109170.pdf" H 5100 7250 30  0001 C CNN
-F 4 "71-CRCW0603-22.1-E3" H 5100 7250 60  0001 C CNN "Mouse PN"
+F 3 "" H 5100 7250 30  0001 C CNN
 	1    5100 7250
 	0    1    1    0
@@
 P 2800 7300
 F 0 "P18" H 2800 7750 50  0000 C CNN
-F 1 "CONN_02X08" V 2800 7300 50  0000 C CNN
+F 1 "CONN_02X10" V 2800 7300 50  0000 C CNN
 F 2 "Pin_Headers:Pin_Header_Straight_2x10" H 2800 6100 60  0001 C CNN
 F 3 "" H 2800 6100 60  0000 C CNN

Commit message: Added learnings from V1.2 build
Parts:
- removed Q13: BSS84, Custom Parts:SOT-23-123, symbol Q_PMOS_GSD
- removed Q15: 2N7000, Custom Parts:SOT-23-123, symbol Q_NMOS_SGD
- removed R65: 2K0, Custom Parts:R_0603_sm, symbol R
- removed U12, U15, U16, U18: SLG59M, Custom Parts:STDFN-4, symbol SLG59M
- added D4: 4148, Custom Parts:Diode_0805_12_SM, symbol D
- added P?: FPC Cable, symbol TEST
- added U12, U15, U16, U18, U25: Si1865DDL, symbol Si1865DDL
- C42: footprint Capacitors_Tantalum_SMD:TantalC_SizeD_EIA-7343_Reflow -> Capacitors_SMD:c_elec_6.3x5.8
- C43, C50: footprint Custom Parts:C_0805_SM -> Custom Parts:C_1206_SM
- P18: Mouse PN 517-929852-01-10-RA -> 649-SFW20R-2STE1LF
- R59, R67, R68, R76: value 0 -> 10K; Mouse PN 71-CRCW0603-0-E3 -> 71-CRCW0603-10k-E3
- R70, R73: value 10K -> 24K; Mouse PN 71-CRCW0603-10k-E3 -> 71-CRCW0603-24k-E3
- R71: value 2K0 -> 10K; Mouse PN 71-CRCW0603-2.0k-E3 -> 71-CRCW0603-10k-E3
- SW2: Mouse PN 506-FSMSM -> PTS645VK58-2-LFS
Connections:
- wire segments 55 -> 124
- no-connect marks 15 -> 17
Other:
- note removed: "Slew Rate is\nControlable"
- moved on the sheet: C65, D15, R66, R69, R70, R71, R73, R74, SW2

Commit message: got bring-up firmware running
chip inits and clears the shift register
Connections:
- wire segments 124 -> 93
Changed lines of the file:
@@
 Connection ~ 1700 1050
 Wire Wire Line
-	2300 1050 2400 1050
-Wire Wire Line
-	2400 1050 2500 1050
+	2300 1050 2500 1050
 Wire Wire Line
 	2400 1050 2400 1100
@@
 5V0_EN
 Wire Wire Line
-	2250 2300 2550 2300
-Wire Wire Line
-	2550 2300 2800 2300
-Wire Wire Line
-	2800 2300 2950 2300
+	2250 2300 2950 2300
 Connection ~ 2550 2300
 Connection ~ 2800 2300
@@
 	2550 2700 2550 2800
 Wire Wire Line
-	2450 2800 2550 2800
-Wire Wire Line
-	2550 2800 2650 2800
+	2450 2800 2650 2800
 Connection ~ 2550 2800
 $Comp
@@
 $EndComp
 Wire Wire Line
-	3150 2800 3250 2800
-Wire Wire Line
-	3250 2800 3450 2800
-Wire Wire Line
-	3450 2800 3700 2800
+	3150 2800 3700 2800
 Wire Wire Line
 	3250 3050 3250 2800
 Wire Wire Line
-	1700 3050 1800 3050
-Wire Wire Line
-	1800 3050 3250 3050
+	1700 3050 3250 3050
 Connection ~ 3250 2800
 Wire Wire Line
@@
 	1400 3050 1350 3050
 Wire Wire Line
-	1350 3050 1350 2800
-Wire Wire Line
-	1250 2800 1300 2800
-Wire Wire Line
-	1300 2800 1350 2800
-Wire Wire Line
-	1350 2800 1400 2800
+	1350 2800 1350 3050
+Wire Wire Line
+	1250 2800 1400 2800
 Connection ~ 1350 2800
 Wire Wire Line
@@
 $EndComp
 Wire Wire Line
-	4350 3950 4650 3950
-Wire Wire Line
-	4650 3950 4900 3950
-Wire Wire Line
-	4900 3950 5050 3950
+	4350 3950 5050 3950
 Connection ~ 4650 3950
 Connection ~ 4900 3950
@@
 	4650 4350 4650 4450
 Wire Wire Line
-	4550 4450 4650 4450
-Wire Wire Line
-	4650 4450 4750 4450
+	4550 4450 4750 4450
 Connection ~ 4650 4450
 Wire Wire Line
 	5350 4700 5350 4450
 Wire Wire Line
-	3800 4700 3900 4700
-Wire Wire Line
-	3900 4700 5350 4700
+	3800 4700 5350 4700
 Connection ~ 5350 4450
 Wire Wire Line
@@
 	3500 4700 3450 4700
 Wire Wire Line
-	3450 4450 3450 4700
-Wire Wire Line
-	3450 4700 3450 4750
+	3450 4450 3450 4750
 Connection ~ 3450 4450
 Wire Wire Line
@@
 3V3_A
 Wire Wire Line
-	5250 4450 5350 4450
-Wire Wire Line
-	5350 4450 5550 4450
+	5250 4450 5550 4450
 $Comp
 L GND #PWR067
@@
 BUTTON
 Wire Wire Line
-	900  5100 1600 5100
-Wire Wire Line
-	1600 5100 1900 5100
-Wire Wire Line
-	1900 5100 1950 5100
+	900  5100 1950 5100
 Wire Wire Line
 	1600 5100 1600 5150
@@
 $EndComp
 Wire Wire Line
-	2550 3950 2650 3950
-Wire Wire Line
-	2650 3950 2800 3950
-Wire Wire Line
-	2800 3950 3450 3950
+	2550 3950 3450 3950
 Connection ~ 2650 3950
 Connection ~ 2800 3950
@@
 Connection ~ 3450 4700
 Wire Wire Line
-	3400 4450 3450 4450
-Wire Wire Line
-	3450 4450 3500 4450
+	3400 4450 3500 4450
 Text Notes 800  6150 0    69   ~ 0
 Button force starts the 3V3 to start SEQ\nSEQ must hold 3V3_EN high to stay on\nBUTTON is soft button signal once running\n3V3_EN pulled low kills supply regaurdless if button pressed
@@
 	5250 7250 5300 7250
 Wire Wire Line
-	5250 7400 5300 7400
-Wire Wire Line
-	5300 7400 5350 7400
+	5250 7400 5350 7400
 Connection ~ 5300 7400
 Text GLabel 3050 7050 2    60   Input ~ 0
@@
 $EndComp
 Wire Wire Line
-	2250 5100 2400 5100
-Wire Wire Line
-	2400 5100 2650 5100
+	2250 5100 2650 5100
 Connection ~ 2400 5100
 $Comp
@@
 	2650 3950 2650 4000
 Wire Wire Line
-	2150 3950 2200 3950
-Wire Wire Line
-	2200 3950 2250 3950
+	2150 3950 2250 3950
 Wire Wire Line
 	2200 3950 2200 4050
@@
 $EndComp
 Wire Wire Line
-	6400 4000 6500 4000
-Wire Wire Line
-	6500 4000 6600 4000
+	6400 4000 6600 4000
 Wire Wire Line
 	6500 4000 6500 4100
@@
 	6550 4500 6600 4500
 Wire Wire Line
-	7850 4000 7900 4000
-Wire Wire Line
-	7900 4000 7950 4000
+	7850 4000 7950 4000
 Wire Wire Line
 	7900 4000 7900 4100
@@
 $EndComp
 Wire Wire Line
-	8300 4350 8400 4350
-Wire Wire Line
-	8400 4350 8500 4350
+	8300 4350 8500 4350
 Wire Wire Line
 	8400 4350 8400 4450
@@
 	8450 4850 8500 4850
 Wire Wire Line
-	9750 4350 9800 4350
-Wire Wire Line
-	9800 4350 9850 4350
+	9750 4350 9850 4350
 Wire Wire Line
 	9800 4350 9800 4450
@@
 $EndComp
 Wire Wire Line
-	6800 5450 6900 5450
-Wire Wire Line
-	6900 5450 7000 5450
+	6800 5450 7000 5450
 Wire Wire Line
 	6900 5450 6900 5550
@@
 	6950 5950 7000 5950
 Wire Wire Line
-	8250 5450 8300 5450
-Wire Wire Line
-	8300 5450 8350 5450
+	8250 5450 8350 5450
 Wire Wire Line
 	8300 5450 8300 5550
@@
 $EndComp
 Wire Wire Line
-	6150 2200 6200 2200
-Wire Wire Line
-	6200 2200 6250 2200
+	6150 2200 6250 2200
 Wire Wire Line
 	6200 2200 6200 2300
@@
 Connection ~ 6200 2200
 Wire Wire Line
-	4750 2200 4800 2200
-Wire Wire Line
-	4800 2200 4900 2200
+	4750 2200 4900 2200
 Wire Wire Line
 	4900 2450 4850 2450

Commit message: V2X Build learnings
Parts:
- P18: Mouse PN 649-SFW20R-2STE1LF -> 571-2-84952-0
- R69: value 2K0 -> 10K; Mouse PN 71-CRCW0603-2.0k-E3 -> 71-CRCW0603-10K-E3
- SW2: Mouse PN PTS645VK58-2-LFS -> PTS645VK39-2-LFS
- U12, U15, U18, U25: footprint (none) -> TO_SOT_Packages_SMD:SC-70-6
- U16: footprint (none) -> TO_SOT_Packages_SMD:SC-70-6; Mouse PN (none) -> 78-SI1865DDL-T1-GE3
- gave numbers to parts that had none: 1
Connections:
- wire segments 93 -> 76
Other:
- moved on the sheet: R59, R67, R68, R69, R76, U15, U16, U18, U25
