File: Hardware/Make Files/Active/V2X_PWR.sch (KiCad schematic (older format))
At the start: 65 parts, among them P10 Board Mount 2, P11 Ficudial2, P12 Board Mount 3, P13 Ficudial3, P15 Board Mount 4, P16 Ficudial4, P17 CUR_SEN, P18 CONN_02X10, P19 CUR_SEN, P25 Ficudial1, P27 Ficudial2, P28 Ficudial3, P29 Ficudial4, P30 FPC Cable, P6 Board Mount 1, P7 Ficudial1, P8 USB_A, P9 USB_u, Q11 IRF9335, Q14 IRF9335, SW2 SW_PUSH, U11 XRP6124, U12 Si1865DDL, U15 Si1865DDL, U16 Si1865DDL, U17 XRP6124, U18 Si1865DDL, U25 Si1865DDL

Commit message: 53534 New design verified
Parts:
- removed C50: 4U7, Custom Parts:C_1206_SM, symbol C
- removed C51: 560P, Custom Parts:C_0603_SM, symbol C
- removed C52: 10U, Custom Parts:C_1206_SM, symbol C
- removed D14: SBR3U30P1-7, Diodes_SMD:SOD-123, symbol D_Schottky_Small
- removed D15: MMSZ4678T1G, Diodes_SMD:SOD-123, symbol ZENER
- removed L5: 10U, Custom Parts:4.5x4.5mm_Ind, symbol INDUCTOR_SMALL
- removed P17, P19: CUR_SEN, Connect:PINHEAD1-2, symbol CONN_01X02
- removed P18: CONN_02X10, Pin_Headers:Pin_Header_Straight_2x10, symbol CONN_02X10
- removed P30: FPC Cable, symbol TEST
- removed P9: USB_u, Custom Parts:USB_Micro-B-DX4R005JJ2R1800, symbol USB_OTG
- removed Q14: IRF9335, Custom Parts:SOIC-8_MOS, symbol Q_PMOS_GSD
- removed R10: DNS, Custom Parts:R_0603_sm, symbol R
- removed R11: 0, Custom Parts:R_0603_sm, symbol R
- removed R67, R68, R76: 10K, Custom Parts:R_0603_sm, symbol R
- removed R72: 6K2, Custom Parts:R_0603_sm, symbol R
- removed R75: 2K0, Custom Parts:R_0603_sm, symbol R
- removed U12, U15, U16, U18: Si1865DDL, TO_SOT_Packages_SMD:SC-70-6, symbol Si1865DDL
- removed U17: XRP6124, Housings_SOT-23_SOT-143_TSOT-6:SOT-23-5, symbol XRP6124
- added C14, C21: 220U, Capacitors_SMD:c_elec_6.3x5.8, symbol CP
- added C16, C23, C27: 4U7, CustomParts:C_0805_SM, symbol C
- added C18, C25, C29, C32, C39, C40: 100N, CustomParts:C_0603_SM, symbol C
- added C22: 10N, CustomParts:C_0603_SM, symbol C
- added C26: 330P, CustomParts:C_0603_SM, symbol C
- added C28: 4U7, CustomParts:C_1206_SM, symbol C
- added C30, C31: 10U, CustomParts:C_1206_SM, symbol C
- added D10: SBR3U30P1-7, CustomParts:SOD-123, symbol D_Schottky_Small
- added FB2: 220, CustomParts:R_0603_sm, symbol FILTER
- added L2: 5U6, CustomParts:L_4.5x4.5, symbol INDUCTOR_SMALL
- added Q12: IRF9335, CustomParts:SOIC-8_MOS, symbol Q_PMOS_GSD
- added R45: 2K0, CustomParts:R_0603_sm, symbol R
- added R47: 8K2, CustomParts:R_0603_sm, symbol R
- added U10: FDC6326L, TO_SOT_Packages_SMD:SOT-23-6, symbol Si1865DDL
- added U11, U12, U13: TLV70012DCK, TO_SOT_Packages_SMD:SOT-23-5, symbol TLV70012DCK
- added U9: XRP6124, TO_SOT_Packages_SMD:SOT-23-5, symbol XRP6124
- C13: renamed from C41; footprint Custom Parts:C_0603_SM -> CustomParts:C_0603_SM
- C15: renamed from C44; footprint Custom Parts:C_0603_SM -> CustomParts:C_0603_SM
- C17: renamed from C65; footprint Custom Parts:C_0603_SM -> CustomParts:C_0603_SM
- C20: renamed from C43; footprint Custom Parts:C_1206_SM -> CustomParts:C_1206_SM
- C24: renamed from C45; footprint Custom Parts:C_1206_SM -> CustomParts:C_1206_SM
- D8: renamed from D12; footprint Diodes_SMD:SOD-123 -> CustomParts:SOD-123
- D9: renamed from D4; footprint Custom Parts:Diode_0805_12_SM -> CustomParts:Diode_0805_12_SM
- L1: renamed from L3; footprint Custom Parts:4.5x4.5mm_Ind -> CustomParts:L_4.5x4.5
- P12: renamed from P25; footprint Fiducials:Fiducial_1mm_Dia_2.54mm_Outer_CopperTop -> Fiducials:Fiducial_1mm_Dia_2.54mm_Outer_CopperBottom
- P13: renamed from P27; footprint Fiducials:Fiducial_1mm_Dia_2.54mm_Outer_CopperTop -> Fiducials:Fiducial_1mm_Dia_2.54mm_Outer_CopperBottom
- P14: renamed from P28; footprint Fiducials:Fiducial_1mm_Dia_2.54mm_Outer_CopperTop -> Fiducials:Fiducial_1mm_Dia_2.54mm_Outer_CopperBottom
- P15: renamed from P29; footprint Fiducials:Fiducial_1mm_Dia_2.54mm_Outer_CopperTop -> Fiducials:Fiducial_1mm_Dia_2.54mm_Outer_CopperBottom
- P3: renamed from P8; footprint Connect:USB_A -> CustomParts:USB-A-SMT; Mouse PN 523-UE27AC5410H -> 806-KUSSMT2AS1NBTR
- Q11: footprint Custom Parts:SOIC-8_MOS -> CustomParts:SOIC-8_MOS
- R37: renamed from R69; footprint Custom Parts:R_0603_sm -> CustomParts:R_0603_sm
- R38: renamed from R73; footprint Custom Parts:R_0603_sm -> CustomParts:R_0603_sm
- R39: renamed from R61; footprint Custom Parts:R_0603_sm -> CustomParts:R_0603_sm
- R40: renamed from R62; footprint Custom Parts:R_0603_sm -> CustomParts:R_0603_sm
- R41: renamed from R71; footprint Custom Parts:R_0603_sm -> CustomParts:R_0603_sm; Mouse PN 71-CRCW0603-10k-E3 -> 71-CRCW0603-10K-E3
- R42: renamed from R66; footprint Custom Parts:R_0603_sm -> CustomParts:R_0603_sm
- R43: renamed from R74; footprint Custom Parts:R_0603_sm -> CustomParts:R_0603_sm
- R44: renamed from R70; footprint Custom Parts:R_0603_sm -> CustomParts:R_0603_sm
- R46: renamed from R59; footprint Custom Parts:R_0603_sm -> CustomParts:R_0603_sm
- R51: renamed from R88; footprint Custom Parts:R_0603_sm -> CustomParts:R_0603_sm
- R52: renamed from R89; footprint Custom Parts:R_0603_sm -> CustomParts:R_0603_sm
- SW2: footprint Custom Parts:PTS645VK58-2-LFS -> CustomParts:PTS645VK58-2-LFS
- U7: renamed from U25; value Si1865DDL -> FDC6326L; footprint TO_SOT_Packages_SMD:SC-70-6 -> TO_SOT_Packages_SMD:SOT-23-6
- U8: renamed from U11; footprint Housings_SOT-23_SOT-143_TSOT-6:SOT-23-5 -> TO_SOT_Packages_SMD:SOT-23-5
- renumbered C42 to C19, D11 to D6, D10 to D7, P13 to P10, P16 to P11, P6 to P4, P10 to P5, P12 to P6, P15 to P7, P7 to P8, P11 to P9
Connections:
- net 12V0_B: now also C28.1, C39.1, Q12.2 (S), U13.1 (IN), U9.5 (VIN)
- net 3V3_EN: now also U13.3 (EN); no longer D9.2 (A)
- net 4V1_EN: now also D9.2 (A)
- net 5V0_A: now also C15.1, C24.1, L1.2, R40.2, U10.4 (S2)
- net 5V0_B: now also U10.2 (D2), U10.3 (D2)
- net 5V0_B_EN: now also U10.5 (EN)
- net GND: now also C14.2, C16.2, C18.2, C21.2, C22.2, C23.2, C25.2, C27.2, C28.2, C29.2, C30.2, C31.2, C32.2, C39.2, C40.2, D10.2 (A), R45.1, U10.1 (R2), U11.2 (GND), U12.2 (GND), U13.2 (GND), U9.2 (GND)
- net at D9.1 (K), R42.1, R44.2: now also U9.1 (EN)
- net at R46.2: now also U10.6 (R1C1)
- new net: C26.2, R45.2, R47.2, U9.3 (FB)
- new net: D10.1 (K), L2.1, Q12.3 (D)
- new net: Q12.1 (G), U9.4 (GATE)
- new net 3V3: C32.1, C40.1, U12.5 (OUT), U13.5 (OUT)
- new net 3V3F1: C27.1, U11.5 (OUT)
- new net 4V1: C14.1, C16.1, C18.1, C26.1, C29.1, C30.1, C31.1, FB2.2, L2.2, R47.1, U12.1 (IN), U12.3 (EN)
- new net 4V1F1: C21.1, C22.1, C23.1, C25.1, FB2.1, U11.1 (IN)
- new net GPS_EN: U11.3 (EN)
- no-connect marks 17 -> 14
Other:
- note added: "4.1V @ 1.5A DC-DC Power Supply"
- note added: "5V @ 1A DC-DC Power Supply"
- note added: "Button starts the 4V1 -> 3V3 supplies\nMust hold 4V1_EN high to stay on\nBUTTON is input signal once running"
- note removed: "3.3V @ 1A DC-DC Power Supply"
- note removed: "5V @ 1.25A DC-DC Power Supply"
- note removed: "Accelerometer 3V3 rail"
- note removed: "Button force starts the 3V3 to start SEQ\nSEQ must hold 3V3_EN high to stay on\nBUTTON is soft button signal once running\n3V3_EN pulled low kills supply regaurdless if button pressed"
- note removed: "CAN 3V3 rail"
- note removed: "GSM+GPS board header"
- note removed: "HUB & FTDI 3V3 rail"
- note removed: "HUB Data, HOST Power"
- note removed: "SEQ side"
- note removed: "SEQ will disable the 3V3 Supply\nand siphon power from 4V1 while \nin SMS standby recieve power state."
- moved on the sheet: C13, C15, C17, C19, C20, C24, D6, D7, D8, D9, F1, F2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
