File: Hardware/Make Files/Active/V2X_GSM.sch (KiCad schematic (older format))
At the start: 42 parts, among them P1 SIM_SKT, P14 CUR_SEN, P2 SMA, P26 CONN_02X10, P3 SMA, Q12 IRF9335, U13 XRP6124, U24 TLV70012DCK, U3 MMQA5V6T3G, U4 SIM5320

Commit message: 53534 New design verified
Parts:
- removed C15, C46: 330P, Custom Parts:C_0603_SM, symbol C
- removed C19, C25: 100N, Custom Parts:C_0603_SM, symbol C
- removed C20, C24, C28: 4U7, Custom Parts:C_0805_SM, symbol C
- removed C23, C26: 220U, Capacitors_SMD:c_elec_6.3x5.8, symbol CP
- removed C27: 10N, Custom Parts:C_0603_SM, symbol C
- removed C47: 4U7, Custom Parts:C_1206_SM, symbol C
- removed C48, C49: 10U, Custom Parts:C_1206_SM, symbol C
- removed D3: SBR3U30P1-7, Diodes_SMD:SOD-123, symbol D_Schottky_Small
- removed FB3: 220, Custom Parts:R_0603_sm, symbol FILTER
- removed L4: 5U6, Custom Parts:4.5x4.5mm_Ind, symbol INDUCTOR_SMALL
- removed P14: CUR_SEN, Connect:PINHEAD1-2, symbol CONN_01X02
- removed P26: CONN_02X10, Pin_Headers:Pin_Header_Straight_2x10, symbol CONN_02X10
- removed Q12: IRF9335, Custom Parts:SOIC-8_MOS, symbol Q_PMOS_GSD
- removed R16: 2K0, Custom Parts:R_0603_sm, symbol R
- removed R17: 8K2, Custom Parts:R_0603_sm, symbol R
- removed R84, R86: DNS, Custom Parts:R_0603_sm, symbol R
- removed R85: 0, Custom Parts:R_0603_sm, symbol R
- removed U13: XRP6124, Housings_SOT-23_SOT-143_TSOT-6:SOT-23-5, symbol XRP6124
- removed U24: TLV70012DCK, TO_SOT_Packages_SMD:SOT-23-5, symbol TLV70012DCK
- C48: renamed from C17; footprint Custom Parts:C_0603_SM -> CustomParts:C_0603_SM
- C49: renamed from C14; footprint Custom Parts:C_0603_SM -> CustomParts:C_0603_SM
- C50: renamed from C18; footprint Custom Parts:C_0603_SM -> CustomParts:C_0603_SM
- C51: renamed from C21; footprint Custom Parts:C_0603_SM -> CustomParts:C_0603_SM
- L3: renamed from L2; footprint Custom Parts:C_0603_SM -> CustomParts:L_0603_SM
- L4: renamed from L1; footprint Custom Parts:C_0603_SM -> CustomParts:L_0603_SM
- P22: renamed from P2; footprint Custom Parts:SMA-RA_142-0701-801 -> CustomParts:SMA-RA_142-0701-801
- P23: renamed from P3; footprint Custom Parts:SMA-RA_142-0701-801 -> CustomParts:SMA-RA_142-0701-801
- P24: renamed from P1; footprint Custom Parts:47553-1001 -> CustomParts:47553-1001
- R69: renamed from R13; footprint Custom Parts:R_0603_sm -> CustomParts:R_0603_sm
- R70: renamed from R12; footprint Custom Parts:R_0603_sm -> CustomParts:R_0603_sm
- R71: renamed from R14; footprint Custom Parts:R_0603_sm -> CustomParts:R_0603_sm
- U22: renamed from U4; footprint Custom Parts:SIM5320 -> CustomParts:SIM5320
- U23: renamed from U3; footprint Housings_SOT-23_SOT-143_TSOT-6:SOT-23-6 -> TO_SOT_Packages_SMD:SOT-23-6
- renumbered C16 to C47, W2 to W1
Connections:
- net 4V1_B renamed 4V1
- net PC_WAKE renamed SEQ_WAKE
- net SIMCARD_B renamed SIMCARD
- net SIM_DM_B renamed SIM_DM
- net SIM_DP_B renamed SIM_DP
- net SIM_DTR: no longer names the net of U22.72 (UART_DTR)
- net SIM_NET_B renamed SIM_NET
- net SIM_PWR_B renamed GPS_EN
- net SIM_PWR_ON_B renamed ~SIM_PWR_ON
- net SIM_RESET_B renamed SIM_RESET
- net SIM_RF_OFF_B: no longer names the net of U22.54 (GPIO_4)
- net SIM_RI: no longer names the net of U22.69 (UART_RI)
- net SIM_RXD_B renamed SIM_RXD
- net SIM_TXD_B renamed SIM_TXD
- net SIM_USB_DET_B renamed HUB_PWR_PRT2
- net SIM_WAKE_B renamed SIM_WAKE
- no-connect marks 38 -> 41
Other:
- note removed: "4.1V @ 1.5A DC-DC Power Supply"
- note removed: "Hopefully the PWRCTRL can \nmomentarily use a pull up \nresistor to snense the card,\n otherwise resistors"
- note removed: "SIM side"
- moved on the sheet: C48, C49, C50, C51, L3, L4, P22, P23, U23, W1
