File: Hardware/Make Files/Active/V2X_OBD.sch (KiCad schematic (older format))
At the start: 79 parts, among them J1 DB9, P4 DB-9 to OBD2, P5 NVM_RST, Q1 2N7000, Q10 2N3904, Q2 BSS84, Q3 BSS84, Q4 BSS84, Q5 3906, Q6 2N3904, Q7 2N7000, Q8 2N3904, Q9 2N3904, SW1 SPST, U10 MCP2551, U5 ESDAxxSC6, U6 ESDAxxSC6, U7 STN1110, U8 LM339, U9 LM317, X2 16MHz

Commit message: Verification findings and modifications
Connections:
- no-connect marks 2 -> 8
Other:
- moved on the sheet: P4
Changed lines of the file:
@@
 J1850_BUS_+_TX
 $Comp
-L GND #PWR41
+L GND #PWR019
 U 1 1 55A9EB78
 P 7100 2050
-F 0 "#PWR41" H 7100 1800 50  0001 C CNN
+F 0 "#PWR019" H 7100 1800 50  0001 C CNN
 F 1 "GND" V 7100 1850 50  0000 C CNN
 F 2 "" H 7100 2050 60  0000 C CNN
@@
 CAN_RX
 $Comp
-L GND #PWR45
+L GND #PWR020
 U 1 1 55A9F1D5
 P 9200 1100
-F 0 "#PWR45" H 9200 850 50  0001 C CNN
+F 0 "#PWR020" H 9200 850 50  0001 C CNN
 F 1 "GND" H 9200 950 50  0000 C CNN
 F 2 "" H 9200 1100 60  0000 C CNN
@@
 $EndComp
 $Comp
-L GND #PWR48
+L GND #PWR021
 U 1 1 55AA095B
 P 10200 2400
-F 0 "#PWR48" H 10200 2150 50  0001 C CNN
+F 0 "#PWR021" H 10200 2150 50  0001 C CNN
 F 1 "GND" H 10200 2250 50  0000 C CNN
 F 2 "" H 10200 2400 60  0000 C CNN
@@
 ISO_K_TX
 $Comp
-L GND #PWR20
+L GND #PWR022
 U 1 1 55AA4905
 P 1550 900
-F 0 "#PWR20" H 1550 650 50  0001 C CNN
+F 0 "#PWR022" H 1550 650 50  0001 C CNN
 F 1 "GND" H 1550 750 50  0000 C CNN
 F 2 "" H 1550 900 60  0000 C CNN
@@
 OBD2 Connector
 $Comp
-L GND #PWR44
+L GND #PWR023
 U 1 1 55AA65C2
 P 8800 1450
-F 0 "#PWR44" H 8800 1200 50  0001 C CNN
+F 0 "#PWR023" H 8800 1200 50  0001 C CNN
 F 1 "GND" V 8800 1250 50  0000 C CNN
 F 2 "" H 8800 1450 60  0000 C CNN
@@
 F 0 "U10" H 5550 6950 50  0000 L CNN
 F 1 "MCP2551" H 6050 6950 50  0000 L CNN
-F 2 "Housings_SOIC:SOIC-8_3.9x4.9mm_Pitch1.27mm" H 5950 6600 50  0000 C CIN
+F 2 "Housings_SOIC:SOIC-8_3.9x4.9mm_Pitch1.27mm" H 5950 6600 50  0001 C CIN
 F 3 "http://www.mouser.com/ds/2/268/21667d-63675.pdf" H 5950 6600 60  0001 C CNN
 F 4 "579-MCP2551-I/SN" H 5950 6600 60  0001 C CNN "Mouse PN"
@@
 NoConn ~ 6450 6700
 $Comp
-L GND #PWR40
+L GND #PWR024
 U 1 1 55B1EF7D
 P 6550 7100
-F 0 "#PWR40" H 6550 6850 50  0001 C CNN
+F 0 "#PWR024" H 6550 6850 50  0001 C CNN
 F 1 "GND" H 6550 6950 50  0000 C CNN
 F 2 "" H 6550 7100 60  0000 C CNN
@@
 $EndComp
 $Comp
-L GND #PWR39
+L GND #PWR025
 U 1 1 55B1F182
 P 5950 7000
-F 0 "#PWR39" H 5950 6750 50  0001 C CNN
+F 0 "#PWR025" H 5950 6750 50  0001 C CNN
 F 1 "GND" H 5950 6850 50  0000 C CNN
 F 2 "" H 5950 7000 60  0000 C CNN
@@
 $EndComp
 $Comp
-L GND #PWR35
+L GND #PWR026
 U 1 1 55B1F6A3
 P 4950 7400
-F 0 "#PWR35" H 4950 7150 50  0001 C CNN
+F 0 "#PWR026" H 4950 7150 50  0001 C CNN
 F 1 "GND" H 4950 7250 50  0000 C CNN
 F 2 "" H 4950 7400 60  0000 C CNN
@@
 $EndComp
 $Comp
-L GND #PWR37
+L GND #PWR027
 U 1 1 55B1F6FC
 P 5250 7400
-F 0 "#PWR37" H 5250 7150 50  0001 C CNN
+F 0 "#PWR027" H 5250 7150 50  0001 C CNN
 F 1 "GND" H 5250 7250 50  0000 C CNN
 F 2 "" H 5250 7400 60  0000 C CNN
@@
 $EndComp
 $Comp
-L GND #PWR22
+L GND #PWR028
 U 1 1 55B20611
 P 1750 7050
-F 0 "#PWR22" H 1750 6800 50  0001 C CNN
+F 0 "#PWR028" H 1750 6800 50  0001 C CNN
 F 1 "GND" H 1750 6900 50  0000 C CNN
 F 2 "" H 1750 7050 60  0000 C CNN
@@
 $EndComp
 $Comp
-L GND #PWR29
+L GND #PWR029
 U 1 1 55B21D3D
 P 3300 7400
-F 0 "#PWR29" H 3300 7150 50  0001 C CNN
+F 0 "#PWR029" H 3300 7150 50  0001 C CNN
 F 1 "GND" H 3300 7250 50  0000 C CNN
 F 2 "" H 3300 7400 60  0000 C CNN
@@
 $EndComp
 $Comp
-L GND #PWR26
+L GND #PWR030
 U 1 1 55B21DB4
 P 2700 7000
-F 0 "#PWR26" H 2700 6750 50  0001 C CNN
+F 0 "#PWR030" H 2700 6750 50  0001 C CNN
 F 1 "GND" V 2700 6800 50  0000 C CNN
 F 2 "" H 2700 7000 60  0000 C CNN
@@
 $EndComp
 $Comp
-L GND #PWR19
+L GND #PWR031
 U 1 1 55B2AD22
 P 1200 4000
-F 0 "#PWR19" H 1200 3750 50  0001 C CNN
+F 0 "#PWR031" H 1200 3750 50  0001 C CNN
 F 1 "GND" H 1200 3850 50  0000 C CNN
 F 2 "" H 1200 4000 60  0000 C CNN
@@
 $EndComp
 $Comp
-L GND #PWR23
+L GND #PWR032
 U 1 1 55B2AE3A
 P 2100 3050
-F 0 "#PWR23" H 2100 2800 50  0001 C CNN
+F 0 "#PWR032" H 2100 2800 50  0001 C CNN
 F 1 "GND" H 2100 2900 50  0000 C CNN
 F 2 "" H 2100 3050 60  0000 C CNN
@@
 $EndComp
 $Comp
-L GND #PWR25
+L GND #PWR033
 U 1 1 55B2EC6D
 P 2450 5450
-F 0 "#PWR25" H 2450 5200 50  0001 C CNN
+F 0 "#PWR033" H 2450 5200 50  0001 C CNN
 F 1 "GND" H 2450 5300 50  0000 C CNN
 F 2 "" H 2450 5450 60  0000 C CNN
@@
 $EndComp
 $Comp
-L GND #PWR24
+L GND #PWR034
 U 1 1 55B36180
 P 2350 4100
-F 0 "#PWR24" H 2350 3850 50  0001 C CNN
+F 0 "#PWR034" H 2350 3850 50  0001 C CNN
 F 1 "GND" H 2350 3950 50  0000 C CNN
 F 2 "" H 2350 4100 60  0000 C CNN
@@
 $EndComp
 $Comp
-L GND #PWR34
+L GND #PWR035
 U 1 1 55B3623F
 P 4800 4550
-F 0 "#PWR34" H 4800 4300 50  0001 C CNN
+F 0 "#PWR035" H 4800 4300 50  0001 C CNN
 F 1 "GND" H 4800 4400 50  0000 C CNN
 F 2 "" H 4800 4550 60  0000 C CNN
@@
 $EndComp
 $Comp
-L GND #PWR38
+L GND #PWR036
 U 1 1 55B362FE
 P 5500 5150
-F 0 "#PWR38" H 5500 4900 50  0001 C CNN
+F 0 "#PWR036" H 5500 4900 50  0001 C CNN
 F 1 "GND" H 5500 5000 50  0000 C CNN
 F 2 "" H 5500 5150 60  0000 C CNN
@@
 $EndComp
 $Comp
-L GND #PWR33
+L GND #PWR037
 U 1 1 55B38770
 P 4600 3250
-F 0 "#PWR33" H 4600 3000 50  0001 C CNN
+F 0 "#PWR037" H 4600 3000 50  0001 C CNN
 F 1 "GND" H 4600 3100 50  0000 C CNN
 F 2 "" H 4600 3250 60  0000 C CNN
@@
 $EndComp
 $Comp
-L GND #PWR32
+L GND #PWR038
 U 1 1 55B3930C
 P 4300 3950
-F 0 "#PWR32" H 4300 3700 50  0001 C CNN
+F 0 "#PWR038" H 4300 3700 50  0001 C CNN
 F 1 "GND" H 4300 3800 50  0000 C CNN
 F 2 "" H 4300 3950 60  0000 C CNN
@@
 CAN_H and CAN_L are high-z until UVLO
 $Comp
-L GND #PWR47
+L GND #PWR039
 U 1 1 55B828E1
 P 9700 3800
-F 0 "#PWR47" H 9700 3550 50  0001 C CNN
+F 0 "#PWR039" H 9700 3550 50  0001 C CNN
 F 1 "GND" H 9700 3650 50  0000 C CNN
 F 2 "" H 9700 3800 60  0000 C CNN
@@
 CAN_3.3V_SW
 $Comp
-L GND #PWR42
+L GND #PWR040
 U 1 1 55B888B6
 P 8100 5200
-F 0 "#PWR42" H 8100 4950 50  0001 C CNN
+F 0 "#PWR040" H 8100 4950 50  0001 C CNN
 F 1 "GND" H 8100 5050 50  0000 C CNN
 F 2 "" H 8100 5200 60  0000 C CNN
@@
 CAN_5V_SW
 $Comp
-L GND #PWR49
+L GND #PWR041
 U 1 1 55B98D87
 P 10300 3800
-F 0 "#PWR49" H 10300 3550 50  0001 C CNN
+F 0 "#PWR041" H 10300 3550 50  0001 C CNN
 F 1 "GND" H 10300 3650 50  0000 C CNN
 F 2 "" H 10300 3800 60  0000 C CNN
@@
 $EndComp
 $Comp
-L GND #PWR50
+L GND #PWR042
 U 1 1 55B98E50
 P 10600 3800
-F 0 "#PWR50" H 10600 3550 50  0001 C CNN
+F 0 "#PWR042" H 10600 3550 50  0001 C CNN
 F 1 "GND" H 10600 3650 50  0000 C CNN
 F 2 "" H 10600 3800 60  0000 C CNN
@@
 CAN_12V_SW
 $Comp
-L GND #PWR46
+L GND #PWR043
 U 1 1 55BC6F4D
 P 9350 3800
-F 0 "#PWR46" H 9350 3550 50  0001 C CNN
+F 0 "#PWR043" H 9350 3550 50  0001 C CNN
 F 1 "GND" H 9350 3650 50  0000 C CNN
 F 2 "" H 9350 3800 60  0000 C CNN
@@
 $EndComp
 $Comp
-L GND #PWR36
+L GND #PWR044
 U 1 1 55BD1D18
 P 5150 1600
-F 0 "#PWR36" H 5150 1350 50  0001 C CNN
+F 0 "#PWR044" H 5150 1350 50  0001 C CNN
 F 1 "GND" H 5150 1450 50  0000 C CNN
 F 2 "" H 5150 1600 60  0000 C CNN
@@
 	10600 3800 10900 3800
 $Comp
-L GND #PWR27
+L GND #PWR045
 U 1 1 55C0BB59
 P 3150 900
-F 0 "#PWR27" H 3150 650 50  0001 C CNN
+F 0 "#PWR045" H 3150 650 50  0001 C CNN
 F 1 "GND" H 3150 750 50  0000 C CNN
 F 2 "" H 3150 900 60  0000 C CNN
@@
 	2550 1300 2550 1600
 $Comp
-L GND #PWR28
+L GND #PWR046
 U 1 1 55C18827
 P 3150 1700
-F 0 "#PWR28" H 3150 1450 50  0001 C CNN
+F 0 "#PWR046" H 3150 1450 50  0001 C CNN
 F 1 "GND" H 3150 1550 50  0000 C CNN
 F 2 "" H 3150 1700 60  0000 C CNN
@@
 	2550 1600 1550 1600
 $Comp
-L GND #PWR21
+L GND #PWR047
 U 1 1 55B3CF26
 P 1550 1100
-F 0 "#PWR21" H 1550 850 50  0001 C CNN
+F 0 "#PWR047" H 1550 850 50  0001 C CNN
 F 1 "GND" H 1550 950 50  0000 C CNN
 F 2 "" H 1550 1100 60  0000 C CNN
@@
 	10550 4250 10500 4250
 $Comp
-L GND #PWR30
+L GND #PWR048
 U 1 1 55B38EC3
 P 3950 900
-F 0 "#PWR30" H 3950 650 50  0001 C CNN
+F 0 "#PWR048" H 3950 650 50  0001 C CNN
 F 1 "GND" H 3950 750 50  0000 C CNN
 F 2 "" H 3950 900 60  0000 C CNN
@@
 $EndComp
 $Comp
-L GND #PWR31
+L GND #PWR049
 U 1 1 55B390EE
 P 3950 1700
-F 0 "#PWR31" H 3950 1450 50  0001 C CNN
+F 0 "#PWR049" H 3950 1450 50  0001 C CNN
 F 1 "GND" H 3950 1550 50  0000 C CNN
 F 2 "" H 3950 1700 60  0000 C CNN
@@
 $EndComp
 $Comp
-L GND #PWR43
+L GND #PWR050
 U 1 1 55B7C569
 P 8100 6150
-F 0 "#PWR43" H 8100 5900 50  0001 C CNN
+F 0 "#PWR050" H 8100 5900 50  0001 C CNN
 F 1 "GND" H 8100 6000 50  0000 C CNN
 F 2 "" H 8100 6150 60  0000 C CNN
@@
 L CONN_01X01 P4
 U 1 1 55B92A71
-P 750 1550
-F 0 "P4" H 750 1650 50  0000 C CNN
-F 1 "DB-9 to OBD2" V 850 1550 50  0000 C CNN
-F 2 "" H 750 1550 60  0001 C CNN
-F 3 "http://www.amazon.com/Adapter-Cable--Connecting-Diagnostic-Interface-Compliant/dp/B007UKTW8E/ref=sr_1_1?ie=UTF8&qid=1443117694&sr=8-1" H 750 1550 60  0001 C CNN
-	1    750  1550
-	1    0    0    -1
-$EndComp
-NoConn ~ 550  1550
+P 10650 1100
+F 0 "P4" H 10650 1200 50  0000 C CNN
+F 1 "DB-9 to OBD2" V 10750 1100 50  0000 C CNN
+F 2 "" H 10650 1100 60  0001 C CNN
+F 3 "http://www.amazon.com/Adapter-Cable--Connecting-Diagnostic-Interface-Compliant/dp/B007UKTW8E/ref=sr_1_1?ie=UTF8&qid=1443117694&sr=8-1" H 10650 1100 60  0001 C CNN
+	1    10650 1100
+	1    0    0    -1
+$EndComp
+NoConn ~ 10450 1100
 Wire Wire Line
 	3950 1550 3950 1300
@@
 Text GLabel 9950 4550 3    60   Input ~ 0
 CAN_TXD
-Entry Bus Bus
-	6700 200  6800 300
 $Comp
 L LM339 U8
@@
 	1    0    0    -1
 $EndComp
+NoConn ~ 8800 1750
+NoConn ~ 8800 1850
+NoConn ~ 8800 1950
+NoConn ~ 3450 5150
+NoConn ~ 3450 4950
+NoConn ~ 4150 5050
 $EndSCHEMATC

Commit message: V2X V1.2 PCB build, with shares
Parts:
- U7: symbol STN1110 -> STN1110-RESCUE-V2X
Connections:
- no-connect marks 8 -> 9
Changed lines of the file:
@@
 $EndDescr
 $Comp
-L STN1110 U7
+L STN1110-RESCUE-V2X U7
 U 1 1 55A9EA92
 P 7550 1750
@@
 NoConn ~ 3450 4950
 NoConn ~ 4150 5050
+NoConn ~ 3150 1850
 $EndSCHEMATC

Commit message: BOM updates
Parts:
- C31: Mouse PN 963-LMK212B7475KG-T -> 581-12063C475KAT2A
- R52, R53: value 100 -> 120; Mouse PN 71-CRCW0603-100-E3 -> 71-CRCW0603-120-E3
Changed lines of the file:
@@
 P 4950 6950
 F 0 "R52" V 5030 6950 50  0000 C CNN
-F 1 "100" V 4950 6950 50  0000 C CNN
+F 1 "120" V 4950 6950 50  0000 C CNN
 F 2 "Custom Parts:R_0603_sm" V 4880 6950 30  0001 C CNN
 F 3 "http://www.vishay.com/doc?20035" H 4950 6950 30  0001 C CNN
-F 4 "71-CRCW0603-100-E3" H 4950 6950 60  0001 C CNN "Mouse PN"
+F 4 "71-CRCW0603-120-E3" H 4950 6950 60  0001 C CNN "Mouse PN"
 	1    4950 6950
 	1    0    0    -1
@@
 F 2 "Custom Parts:C_0805_SM" H 9938 2100 30  0001 C CNN
 F 3 "http://www.yuden.co.jp/productdata/catalog/en/mlcc_all_e.pdf" H 9900 2250 60  0001 C CNN
-F 4 "963-LMK212B7475KG-T" H 9900 2250 60  0001 C CNN "Mouse PN"
+F 4 "581-12063C475KAT2A" H 9900 2250 60  0001 C CNN "Mouse PN"
 	1    9900 2250
 	1    0    0    -1
@@
 P 5250 6950
 F 0 "R53" V 5330 6950 50  0000 C CNN
-F 1 "100" V 5250 6950 50  0000 C CNN
+F 1 "120" V 5250 6950 50  0000 C CNN
 F 2 "Custom Parts:R_0603_sm" V 5180 6950 30  0001 C CNN
 F 3 "http://www.vishay.com/doc?20035" H 5250 6950 30  0001 C CNN
-F 4 "71-CRCW0603-100-E3" H 5250 6950 60  0001 C CNN "Mouse PN"
+F 4 "71-CRCW0603-120-E3" H 5250 6950 60  0001 C CNN "Mouse PN"
 	1    5250 6950
 	1    0    0    -1

Commit message: V2X Build learnings
Parts:
- removed R28, R29: 10K, Custom Parts:R_0603_sm, symbol R
- removed R35, R36, R37: 2K2, Custom Parts:R_0603_sm, symbol R
- added R8: 100K, Custom Parts:R_0603_sm, symbol R
- Q1, Q7: symbol Q_NMOS_SGD -> Q_NMOS_GSD
Connections:
- net 3V3_C: now also R8.1
- net CAN_POWERDOWN: now also Q7.1 (G); no longer Q7.2 (G)
- net GND: now also Q1.2 (S), Q7.2 (S); no longer Q1.1 (S), Q7.1 (S)
- net PWM/~VPW: now also Q1.1 (G); no longer Q1.2 (G)
- net at P5.1 (P1), U7.21 (~OBD_TX_LED/RST_NVM): now also R8.2
- net at Q4.1 (G), R30.2: now also Q2.1 (G), Q3.1 (G), Q7.3 (D)
Other:
- moved on the sheet: R30, R39
Changed lines of the file:
@@
 U 1 1 55B7C06D
 P 8300 3850
-F 0 "Q4" H 8600 3900 50  0000 R CNN
-F 1 "BSS84" H 8850 3800 50  0000 R CNN
+F 0 "Q4" H 8250 4000 50  0000 R CNN
+F 1 "BSS84" H 8350 3650 50  0000 R CNN
 F 2 "Custom Parts:SOT-23-123" H 8500 3950 29  0001 C CNN
 F 3 "http://www.mouser.com/ds/2/149/BSS84-39462.pdf" H 8300 3850 60  0001 C CNN
@@
 Text GLabel 6000 6100 2    60   Input ~ 0
 CAN_5V_SW
-Text GLabel 8550 3650 2    60   Input ~ 0
+Text GLabel 8550 3200 2    60   Input ~ 0
 3V3_C
 Text GLabel 3300 6800 1    60   Input ~ 0
@@
 Text GLabel 6700 4050 3    60   Input ~ 0
 CAN_12V_SW
-$Comp
-L R R35
-U 1 1 55BC4846
-P 6400 4000
-F 0 "R35" V 6480 4000 50  0000 C CNN
-F 1 "2K2" V 6400 4000 50  0000 C CNN
-F 2 "Custom Parts:R_0603_sm" V 6330 4000 30  0001 C CNN
-F 3 "http://www.vishay.com/doc?20035" H 6400 4000 30  0001 C CNN
-F 4 "71-CRCW0603-2.2K-E3" H 6400 4000 60  0001 C CNN "Mouse PN"
-	1    6400 4000
-	1    0    0    -1
-$EndComp
 Text GLabel 4600 2850 0    60   Input ~ 0
 CAN_12V_SW
@@
 	2700 5050 2450 5050
 Wire Wire Line
-	7250 3200 7250 3550
-Wire Wire Line
-	6400 3200 8200 3200
-Wire Wire Line
-	8100 3200 8100 3550
-Connection ~ 7250 3200
-Wire Wire Line
-	7250 4150 7250 4700
-Wire Wire Line
-	6400 4700 8100 4700
-Wire Wire Line
-	8100 4150 8100 4800
-Wire Wire Line
-	8550 3950 8550 3650
-Wire Wire Line
-	8550 3650 8400 3650
+	7250 3850 7250 4700
+Wire Wire Line
+	8100 4700 6400 4700
+Wire Wire Line
+	8100 3600 8100 4800
+Wire Wire Line
+	8550 3200 8550 3400
 Connection ~ 8100 4700
 Wire Wire Line
@@
 	2650 2300 2650 2350
 Wire Wire Line
-	6400 4150 6400 4700
+	6400 4700 6400 3850
 Connection ~ 7250 4700
 Wire Wire Line
-	6400 3200 6400 3550
-Wire Wire Line
-	6700 3650 6700 3200
-Connection ~ 6700 3200
+	6700 3200 6700 3650
 Wire Notes Line
 	9100 2900 9100 5400
@@
 CAN_POWERDOWN is open collector\nneeds pullup to opperate.\nIf jumper is out circuit is just on.
 Wire Wire Line
-	8550 4250 8550 5000
+	8550 3700 8550 5000
 Wire Wire Line
 	10250 4550 10250 4700
@@
 Text GLabel 5500 1000 1    60   Input ~ 0
 3V3_C
-Text GLabel 8200 3200 2    60   Input ~ 0
+Text GLabel 6700 3200 0    60   Input ~ 0
 12V0_B
-Connection ~ 8100 3200
 Text GLabel 7550 3650 1    60   Input ~ 0
 5V0_A
@@
 U 1 1 560520AD
 P 7450 3850
-F 0 "Q3" H 7750 3900 50  0000 R CNN
-F 1 "BSS84" H 8000 3800 50  0000 R CNN
+F 0 "Q3" H 7400 4000 50  0000 R CNN
+F 1 "BSS84" H 7500 3650 50  0000 R CNN
 F 2 "Custom Parts:SOT-23-123" H 7650 3950 29  0001 C CNN
 F 3 "http://www.mouser.com/ds/2/149/BSS84-39462.pdf" H 7450 3850 60  0001 C CNN
@@
 U 1 1 560521FD
 P 6600 3850
-F 0 "Q2" H 6900 3900 50  0000 R CNN
-F 1 "BSS84" H 7150 3800 50  0000 R CNN
+F 0 "Q2" H 6550 4000 50  0000 R CNN
+F 1 "BSS84" H 6650 3650 50  0000 R CNN
 F 2 "Custom Parts:SOT-23-123" H 6800 3950 29  0001 C CNN
 F 3 "http://www.mouser.com/ds/2/149/BSS84-39462.pdf" H 6600 3850 60  0001 C CNN
@@
 $EndComp
 $Comp
-L Q_NMOS_SGD Q7
+L Q_NMOS_GSD Q7
 U 1 1 56052C71
 P 8200 5000
@@
 $EndComp
 $Comp
-L R R28
-U 1 1 56052FD9
-P 6400 3700
-F 0 "R28" V 6480 3700 50  0000 C CNN
-F 1 "10K" V 6400 3700 50  0000 C CNN
-F 2 "Custom Parts:R_0603_sm" V 6330 3700 30  0001 C CNN
-F 3 "http://www.vishay.com/doc?20035" H 6400 3700 30  0001 C CNN
-F 4 "71-CRCW0603-10K-E3" H 6400 3700 60  0001 C CNN "Mouse PN"
-	1    6400 3700
-	1    0    0    -1
-$EndComp
-$Comp
-L R R29
-U 1 1 5605361F
-P 7250 3700
-F 0 "R29" V 7330 3700 50  0000 C CNN
-F 1 "10K" V 7250 3700 50  0000 C CNN
-F 2 "Custom Parts:R_0603_sm" V 7180 3700 30  0001 C CNN
-F 3 "http://www.vishay.com/doc?20035" H 7250 3700 30  0001 C CNN
-F 4 "71-CRCW0603-10K-E3" H 7250 3700 60  0001 C CNN "Mouse PN"
-	1    7250 3700
-	1    0    0    -1
-$EndComp
-$Comp
 L R R30
 U 1 1 560537AD
-P 8100 3700
-F 0 "R30" V 8180 3700 50  0000 C CNN
-F 1 "10K" V 8100 3700 50  0000 C CNN
-F 2 "Custom Parts:R_0603_sm" V 8030 3700 30  0001 C CNN
-F 3 "http://www.vishay.com/doc?20035" H 8100 3700 30  0001 C CNN
-F 4 "71-CRCW0603-10K-E3" H 8100 3700 60  0001 C CNN "Mouse PN"
-	1    8100 3700
+P 8100 3450
+F 0 "R30" V 8180 3450 50  0000 C CNN
+F 1 "10K" V 8100 3450 50  0000 C CNN
+F 2 "Custom Parts:R_0603_sm" V 8030 3450 30  0001 C CNN
+F 3 "http://www.vishay.com/doc?20035" H 8100 3450 30  0001 C CNN
+F 4 "71-CRCW0603-10K-E3" H 8100 3450 60  0001 C CNN "Mouse PN"
+	1    8100 3450
 	1    0    0    -1
 $EndComp
@@
 L R R39
 U 1 1 5605393B
-P 8550 4100
-F 0 "R39" V 8630 4100 50  0000 C CNN
-F 1 "10K" V 8550 4100 50  0000 C CNN
-F 2 "Custom Parts:R_0603_sm" V 8480 4100 30  0001 C CNN
-F 3 "http://www.vishay.com/doc?20035" H 8550 4100 30  0001 C CNN
-F 4 "71-CRCW0603-10K-E3" H 8550 4100 60  0001 C CNN "Mouse PN"
-	1    8550 4100
-	1    0    0    -1
-$EndComp
-$Comp
-L R R36
-U 1 1 56054144
-P 7250 4000
-F 0 "R36" V 7330 4000 50  0000 C CNN
-F 1 "2K2" V 7250 4000 50  0000 C CNN
-F 2 "Custom Parts:R_0603_sm" V 7180 4000 30  0001 C CNN
-F 3 "http://www.vishay.com/doc?20035" H 7250 4000 30  0001 C CNN
-F 4 "71-CRCW0603-2.2K-E3" H 7250 4000 60  0001 C CNN "Mouse PN"
-	1    7250 4000
-	1    0    0    -1
-$EndComp
-$Comp
-L R R37
-U 1 1 56054398
-P 8100 4000
-F 0 "R37" V 8180 4000 50  0000 C CNN
-F 1 "2K2" V 8100 4000 50  0000 C CNN
-F 2 "Custom Parts:R_0603_sm" V 8030 4000 30  0001 C CNN
-F 3 "http://www.vishay.com/doc?20035" H 8100 4000 30  0001 C CNN
-F 4 "71-CRCW0603-2.2K-E3" H 8100 4000 60  0001 C CNN "Mouse PN"
-	1    8100 4000
+P 8550 3550
+F 0 "R39" V 8630 3550 50  0000 C CNN
+F 1 "10K" V 8550 3550 50  0000 C CNN
+F 2 "Custom Parts:R_0603_sm" V 8480 3550 30  0001 C CNN
+F 3 "http://www.vishay.com/doc?20035" H 8550 3550 30  0001 C CNN
+F 4 "71-CRCW0603-10K-E3" H 8550 3550 60  0001 C CNN "Mouse PN"
+	1    8550 3550
 	1    0    0    -1
 $EndComp
@@
 $EndComp
 $Comp
-L Q_NMOS_SGD Q1
+L Q_NMOS_GSD Q1
 U 1 1 560643DB
 P 4200 3750
@@
 NoConn ~ 4150 5050
 NoConn ~ 3150 1850
+$Comp
+L R R8
+U 1 1 5655F6EA
+P 10200 1900
+F 0 "R8" V 10280 1900 50  0000 C CNN
+F 1 "100K" V 10200 1900 50  0000 C CNN
+F 2 "Custom Parts:R_0603_sm" V 10130 1900 30  0001 C CNN
+F 3 "http://www.vishay.com/doc?20035" H 10200 1900 30  0001 C CNN
+F 4 "71-CRCW0603-100K-E3" H 10200 1900 60  0001 C CNN "Mouse PN"
+	1    10200 1900
+	1    0    0    -1
+$EndComp
+Text GLabel 10200 1750 1    60   Input ~ 0
+3V3_C
+Connection ~ 8100 3850
+Wire Wire Line
+	8100 3300 8100 3200
+Wire Wire Line
+	8100 3200 6700 3200
+Wire Wire Line
+	8550 3200 8400 3200
+Wire Wire Line
+	8400 3200 8400 3650
 $EndSCHEMATC
