File: Hardware/Make Files/Active/V2X_OBD.sch (KiCad schematic (older format))
At the start: 75 parts, among them J1 DB9, P4 DB-9 to OBD2, P5 NVM_RST, Q1 2N7000, Q10 2N3904, Q2 BSS84, Q3 BSS84, Q4 BSS84, Q5 3906, Q6 2N3904, Q7 2N7000, Q8 2N3904, Q9 2N3904, SW1 SPST, U10 MCP2551, U5 ESDAxxSC6, U6 ESDAxxSC6, U7 STN1110, U8 LM339, U9 LM317, X2 16MHz

Commit message: 53534 New design verified
Parts:
- C1: renamed from C32; footprint Custom Parts:C_0603_SM -> CustomParts:C_0603_SM
- C10: renamed from C36; footprint Custom Parts:C_0603_SM -> CustomParts:C_0603_SM
- C11: renamed from C37; footprint Custom Parts:C_0603_SM -> CustomParts:C_0603_SM
- C12: renamed from C38; footprint Custom Parts:C_0603_SM -> CustomParts:C_0603_SM
- C2: renamed from C30; footprint Custom Parts:C_0603_SM -> CustomParts:C_0603_SM
- C3: renamed from C39; footprint Custom Parts:C_0603_SM -> CustomParts:C_0603_SM
- C4: renamed from C40; footprint Custom Parts:C_0603_SM -> CustomParts:C_0603_SM
- C5: renamed from C29; footprint Custom Parts:C_0603_SM -> CustomParts:C_0603_SM
- C6: renamed from C33; footprint Custom Parts:C_0603_SM -> CustomParts:C_0603_SM
- C7: renamed from C34; footprint Custom Parts:C_0603_SM -> CustomParts:C_0603_SM
- C8: renamed from C31; footprint Custom Parts:C_0805_SM -> CustomParts:C_0805_SM
- C9: renamed from C35; footprint Custom Parts:C_0603_SM -> CustomParts:C_0603_SM
- D1: renamed from D8; footprint Custom Parts:Diode_0805_12_SM -> CustomParts:Diode_0805_12_SM
- D2: renamed from D1; footprint Custom Parts:Diode_0805_12_SM -> CustomParts:Diode_0805_12_SM
- D3: renamed from D2; footprint Custom Parts:Diode_0805_12_SM -> CustomParts:Diode_0805_12_SM
- D4: renamed from D7; footprint Custom Parts:Diode_0805_12_SM -> CustomParts:Diode_0805_12_SM
- D5: renamed from D9; footprint Custom Parts:Diode_0805_12_SM -> CustomParts:Diode_0805_12_SM
- FB1: renamed from FB4; footprint Custom Parts:R_0603_sm -> CustomParts:R_0603_sm
- J1: footprint Custom Parts:D09P13B4PA00LF -> Custom:DB-9_SMT; symbol DB9 -> DB9_SMT; Mouse PN 649-D09P13B4PA00LF -> 617-09551667812741
- P1: renamed from P5; footprint Custom Parts:R_0603_sm -> CustomParts:R_0603_sm
- Q1: renamed from Q9; footprint Custom Parts:SOT-23-123 -> CustomParts:SOT_23_123
- Q10: renamed from Q4; footprint Custom Parts:SOT-23-123 -> CustomParts:SOT_23_123
- Q2: renamed from Q10; footprint Custom Parts:SOT-23-123 -> CustomParts:SOT_23_123
- Q3: renamed from Q8; footprint Custom Parts:SOT-23-123 -> CustomParts:SOT_23_123
- Q4: renamed from Q1; footprint Custom Parts:SOT-23-123 -> CustomParts:SOT_23_123
- Q5: renamed from Q6; footprint Custom Parts:SOT-23-123 -> CustomParts:SOT_23_123
- Q6: renamed from Q5; footprint Custom Parts:SOT-23-123 -> CustomParts:SOT_23_123
- Q7: renamed from Q2; footprint Custom Parts:SOT-23-123 -> CustomParts:SOT_23_123
- Q8: renamed from Q3; footprint Custom Parts:SOT-23-123 -> CustomParts:SOT_23_123
- Q9: renamed from Q7; footprint Custom Parts:SOT-23-123 -> CustomParts:SOT_23_123
- R1: renamed from R49; footprint Custom Parts:R_1210_SM -> CustomParts:R_1210_SM
- R10: renamed from R46; footprint Custom Parts:R_0603_sm -> CustomParts:R_0603_sm
- R11: renamed from R45; footprint Custom Parts:R_0603_sm -> CustomParts:R_0603_sm
- R12: renamed from R21; footprint Custom Parts:R_0603_sm -> CustomParts:R_0603_sm
- R13: renamed from R56; footprint Custom Parts:R_0603_sm -> CustomParts:R_0603_sm
- R14: renamed from R27; footprint Custom Parts:R_0603_sm -> CustomParts:R_0603_sm
- R15: renamed from R57; footprint Custom Parts:R_0603_sm -> CustomParts:R_0603_sm
- R16: renamed from R50; footprint Custom Parts:R_0603_sm -> CustomParts:R_0603_sm
- R17: renamed from R51; footprint Custom Parts:R_0603_sm -> CustomParts:R_0603_sm
- R18: renamed from R40; footprint Custom Parts:R_0603_sm -> CustomParts:R_0603_sm
- R19: renamed from R31; footprint Custom Parts:R_0603_sm -> CustomParts:R_0603_sm
- R2: renamed from R55; footprint Custom Parts:R_1210_SM -> CustomParts:R_1210_SM
- R20: renamed from R24; footprint Custom Parts:R_0603_sm -> CustomParts:R_0603_sm
- R21: renamed from R38; footprint Custom Parts:R_0603_sm -> CustomParts:R_0603_sm
- R22: renamed from R52; footprint Custom Parts:R_0603_sm -> CustomParts:R_0603_sm
- R23: renamed from R32; footprint Custom Parts:R_0603_sm -> CustomParts:R_0603_sm
- R24: renamed from R15; footprint Custom Parts:R_0603_sm -> CustomParts:R_0603_sm
- R25: renamed from R20; footprint Custom Parts:R_0603_sm -> CustomParts:R_0603_sm
- R26: renamed from R53; footprint Custom Parts:R_0603_sm -> CustomParts:R_0603_sm
- R27: renamed from R25; footprint Custom Parts:R_0603_sm -> CustomParts:R_0603_sm
- R28: renamed from R44; footprint Custom Parts:R_0603_sm -> CustomParts:R_0603_sm
- R29: renamed from R54; footprint Custom Parts:R_0603_sm -> CustomParts:R_0603_sm
- R3: renamed from R26; footprint Custom Parts:R_0603_sm -> CustomParts:R_0603_sm
- R30: footprint Custom Parts:R_0603_sm -> CustomParts:R_0603_sm
- R31: renamed from R39; footprint Custom Parts:R_0603_sm -> CustomParts:R_0603_sm
- R32: renamed from R41; footprint Custom Parts:R_0603_sm -> CustomParts:R_0603_sm
- R33: renamed from R8; footprint Custom Parts:R_0603_sm -> CustomParts:R_0603_sm
- R34: renamed from R42; footprint Custom Parts:R_0603_sm -> CustomParts:R_0603_sm
- R35: renamed from R43; footprint Custom Parts:R_0603_sm -> CustomParts:R_0603_sm
- R36: renamed from R47; footprint Custom Parts:R_0603_sm -> CustomParts:R_0603_sm
- R4: renamed from R33; footprint Custom Parts:R_0603_sm -> CustomParts:R_0603_sm
- R5: renamed from R48; footprint Custom Parts:R_0603_sm -> CustomParts:R_0603_sm
- R6: renamed from R58; footprint Custom Parts:R_0603_sm -> CustomParts:R_0603_sm
- R7: renamed from R22; footprint Custom Parts:R_0603_sm -> CustomParts:R_0603_sm
- R8: renamed from R23; footprint Custom Parts:R_0603_sm -> CustomParts:R_0603_sm
- R9: renamed from R34; footprint Custom Parts:R_0603_sm -> CustomParts:R_0603_sm
- SW1: footprint Custom Parts:SW_SPST_FSMSM_SM -> CustomParts:SW_SPST_FSMSM_SM
- U2: renamed from U5; footprint Housings_SOT-23_SOT-143_TSOT-6:SOT-23-6 -> TO_SOT_Packages_SMD:SOT-23-6
- U3: renamed from U6; footprint Housings_SOT-23_SOT-143_TSOT-6:SOT-23-6 -> TO_SOT_Packages_SMD:SOT-23-6
- X1: renamed from X2; footprint Custom Parts:AWSCR -> CustomParts:AWSCR
- renumbered P4 to P2, U8 to U1, U9 to U4, U10 to U5, U7 to U6
Connections:
- net labels added: 3V3
- net labels removed: 3V3_C
- wire segments 105 -> 101
- no-connect marks 9 -> 6
Other:
- moved on the sheet: P2, U1D
