File: Hardware/Make Files/Active/GSM/V2X_GSM.sch (KiCad schematic (older format))
At the start: 46 parts, among them P1 47553-1001, P18 CUR_SEN, P2 SMA, P26 CONN_02X08, P3 SMA, Q12 IRF9335, U14 XRP6124, U3 MMQA5V6T3G, U4 SIM5320

Commit message: V2X V1.2 PCB build, with shares
Parts:
- renumbered C47 to C46, C46 to C47, D13 to D3, P18 to P14, R63 to R16, R64 to R17, U14 to U13
Connections:
- net GND: no longer P26.2 (P2)
- net SIM_WAKE renamed SIM_WAKE_B
- net SIM_WAKE_B: now also P26.2 (P2)
Other:
- moved on the sheet: C23, C24, C25, C26, C27, C28, FB3, P26, R84, R85, R86

Commit message: V1.2 Ordered
This is a capture of the project folder at the time f ordering the V1.2
kit.
Parts:
- removed C22: 47p, Custom Parts:C_0603_SM, symbol C
- removed L6, L7: 47N, Custom Parts:C_0603_SM, symbol INDUCTOR_SMALL
- added U24: TLV70012DCK, Housings_SOT-23_SOT-143_TSOT-6:SOT-23-5, symbol TLV70012DCK
- C15: Mouse PN 77-VJ0603A331FXXCB -> 80-C0603C331J5G
- C17: value 330P -> 56P; Mouse PN 77-VJ0603A331FXXCB -> 581-08052U560G
- C18: value 10N -> 470P; Mouse PN 77-VJ0603Y103KXACBC -> 77-VJ0603D471KXXAJ
- C19: value 330P -> 100N; Mouse PN 77-VJ0603A331FXXCB -> 810-C1608X7R1E104K
- C20: value 10N -> 4U7; footprint Custom Parts:C_0603_SM -> Custom Parts:C_0805_SM; Mouse PN 77-VJ0603Y103KXACBC -> 581-12063C475KAT2A
- C21: value 47p -> 150p; Mouse PN (none) -> 77-VJ0805Q151JXAAC
- C24, C28: Mouse PN 963-LMK212B7475KG-T -> 581-12063C475KAT2A
- L1: value 47N -> 330N
- L2: value 47N -> 120N; Mouse PN 81-LQG18HN47NJ00D -> 81-LQW18CNR12J00D
- P1: value 47553-1001 -> SIM_SKT
- P26: value CONN_02X08 -> CONN_02X10
Connections:
- net GSM is gone; now on net GSM_ANT: P3.1 (P1)
- net 4V1F1: now also C19.1, U24.1 (IN), U24.3 (EN); no longer L1.1
- net GND: now also C17.2, C19.2, U24.2 (GND); no longer C17.1, C19.1
- net at C18.1, L1.2, L2.2: now also C17.1; no longer C17.2
- net 3V3F1: now reaches C20.1
- net 3V3F1: now also L1.1, U24.5 (OUT); no longer C19.2
Other:
- moved on the sheet: C17, C18, C21, L1, L2, P2, P3
