File: Hardware/Make Files/Active/GSM/V2X_GSM.sch (KiCad schematic (older format))
At the start: 43 parts, among them P1 SIM_SKT, P2 SMA, P26 CONN_02X10, P3 SMA, Q12 IRF9335, U13 XRP6124, U24 TLV70012DCK, U3 MMQA5V6T3G, U4 SIM5320

Commit message: part of GSM board update
unsaved files
Parts:
- P26: footprint Pin_Headers:Pin_Header_Straight_2x10 -> Custom Parts:FFC-1MMx20
Connections:
- net 12V0_C: now also P26.19 (P19), P26.20 (P20); no longer P26.1 (P1), P26.2 (P2)
- net 4V1_B: now also P26.15 (P15); no longer P26.6 (P6)
- net 4V1_EN_B: now also P26.16 (P16); no longer P26.5 (P5)
- net GND: now also P26.1 (P1), P26.17 (P17), P26.18 (P18); no longer P26.20 (P20), P26.3 (P3), P26.4 (P4)
- net SIMCARD_B: now also P26.3 (P3); no longer P26.18 (P18)
- net SIM_DM_B: now also P26.7 (P7); no longer P26.14 (P14)
- net SIM_DP_B: now also P26.9 (P9); no longer P26.12 (P12)
- net SIM_NET_B: now also P26.12 (P12); no longer P26.9 (P9)
- net SIM_PWR_B: now also P26.14 (P14); no longer P26.7 (P7)
- net SIM_PWR_ON_B: now also P26.6 (P6); no longer P26.15 (P15)
- net SIM_RESET_B: now also P26.8 (P8); no longer P26.13 (P13)
- net SIM_RF_OFF_B: now also P26.4 (P4); no longer P26.17 (P17)
- net SIM_RXD_B: now also P26.11 (P11); no longer P26.10 (P10)
- net SIM_TXD_B: now also P26.13 (P13); no longer P26.8 (P8)
- net SIM_USB_DET_B: now also P26.5 (P5); no longer P26.16 (P16)
- net SIM_WAKE_B: now also P26.2 (P2); no longer P26.19 (P19)
- net at R84.1, R85.1, R86.1: now also P26.10 (P10); no longer P26.11 (P11)
Changed lines of the file:
@@
 F 0 "P26" H 2200 5550 50  0000 C CNN
 F 1 "CONN_02X10" V 2200 5100 50  0000 C CNN
-F 2 "Pin_Headers:Pin_Header_Straight_2x10" H 2200 3900 60  0001 C CNN
+F 2 "Custom Parts:FFC-1MMx20" H 2200 3900 60  0001 C CNN
 F 3 "http://www.mouser.com/ProductDetail/FCI/77313-824-20LF/?qs=sGAEpiMZZMs%252bGHln7q6pm24n0txessAMJKIe4p3QHSo%3d" H 2200 3900 60  0001 C CNN
 F 4 "649-77313-824-20LF" H 2200 5100 60  0001 C CNN "Mouse PN"
 	1    2200 5100
-	-1   0    0    1
+	1    0    0    -1
 $EndComp
 Text GLabel 1950 4850 0    60   Input ~ 0
